File: schem/pcb/trs_midi_output_8x.sch (KiCad schematic (older format))
At the start: 56 parts

Commit message: First attempts at a PCB layout...
Parts:
- D301, D302, D303, D304, D305, D306, D307, D308, D309, D310, D311, D312, D313, D314, D315, D316: renamed from D?; footprint (none) -> LED_THT:LED_D3.0mm_Horizontal_O6.35mm_Z2.0mm
- J301, J302, J303, J304, J305, J306, J307, J308: renamed from J?; footprint (none) -> Connector_Audio:Jack_3.5mm_Ledino_KB3SPRS_Horizontal
- R301, R302, R303, R304, R305, R306, R307, R308, R309, R310, R311, R312, R313, R314, R315, R316, R317, R318, R319, R320, R321, R322, R323, R324, R325, R326, R327, R328, R329, R330, R331, R332: renamed from R?; footprint (none) -> Resistor_SMD:R_0805_2012Metric
