File: schem/pcb/trsmidi_input_8x.sch (KiCad schematic (older format))
At the start: 56 parts, among them J201 AudioJack3, J202 AudioJack3, J203 AudioJack3, J204 AudioJack3, J205 AudioJack3, J206 AudioJack3, J207 AudioJack3, J208 AudioJack3, U201 HCPL-2630, U202 HCPL-2630, U203 HCPL-2630, U204 HCPL-2630, U205 HCPL-2630, U206 HCPL-2630, U207 HCPL-2630, U208 HCPL-2630

Commit message: First attempts at a PCB layout...
Parts:
- C201, C202, C203, C204, C205, C206, C207, C208: footprint (none) -> Capacitor_SMD:C_0805_2012Metric
- D201, D202, D203, D204, D205, D206, D207, D208: footprint (none) -> LED_THT:LED_D3.0mm_Horizontal_O6.35mm_Z2.0mm
- J201, J202, J203, J204, J205, J206, J207, J208: footprint (none) -> Connector_Audio:Jack_3.5mm_Ledino_KB3SPRS_Horizontal
- R201, R202, R203, R204, R205, R206, R207, R208, R209, R210, R211, R212, R213, R214, R215, R216, R217, R218, R219, R220, R221, R222, R223, R224: footprint (none) -> Resistor_SMD:R_0805_2012Metric
