File: schem/din5_pcb/din5_pcb.kicad_pcb (KiCad board)
At the start: 2 copper layers, 66 parts, among them J1 Conn_01x03_Male, J101 DIN-5_180degree, J102 DIN-5_180degree, J103 DIN-5_180degree, J104 DIN-5_180degree, J2 2x3 female, J201 DIN-5_180degree, J202 DIN-5_180degree, J203 DIN-5_180degree, J204 DIN-5_180degree, J3 2x3 female, U1 74HCT245, U101 HCPL-2630, U102 HCPL-2630, U2 74HC595, U3 74HC165

Commit message: din5 board layout
Parts:
- removed JP10, JP11, JP12, JP13: SolderJumper_2_Open, Jumper:SolderJumper-2_P1.3mm_Open_TrianglePad1.0x1.5mm
- C101, C102, JP1, JP14, JP2, JP3, JP4, R1, R101, R102, R103, R104, R105, R106, R107, R108, R109, R110, R111, R112, R201, R202, R203, R204, R205, R206, R207, R208, R209, R210, R211, R212: moved to B.Cu
- JP5, JP6, JP7, JP8: value SolderJumper_2_Open -> SolderJumper_3_Open; footprint Jumper:SolderJumper-2_P1.3mm_Open_TrianglePad1.0x1.5mm -> Jumper:SolderJumper-3_P1.3mm_Open_RoundedPad1.0x1.5mm; moved to B.Cu
- moved R202 275.9 mm to (22.1, 89.0)
- moved R102 270.1 mm to (25.1, 77.5)
- moved R210 269.8 mm to (25.1, 103.0), turned to 180 degrees
- moved JP4 258.1 mm to (22.5, 24.5), turned to 270 degrees
- moved R209 256.0 mm to (25.1, 52.0), turned to 180 degrees
- moved JP6 254.7 mm to (42.0, 53.5)
- moved R206 253.6 mm to (25.1, 93.0), turned to 180 degrees
- moved R205 250.0 mm to (25.1, 43.7), turned to 180 degrees
- moved JP7 249.7 mm to (42.0, 51.0)
- moved R1 246.3 mm to (48.9, 98.5)
- moved JP5 243.7 mm to (42.0, 56.0)
- moved JP3 239.7 mm to (23.0, 73.8), turned to 270 degrees
- moved R104 237.3 mm to (59.0, 43.0), turned to 180 degrees
- moved R103 236.0 mm to (58.9, 93.0), turned to 180 degrees
- moved R212 233.2 mm to (58.9, 18.0)
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Connections:
- A1 pad PB6: Net-(A1-PadPB6) -> PB6
- A1 pad PB7: Net-(A1-PadPB7) -> PB7
- A1 pad PB8: Net-(A1-PadPB8) -> PB8
- A1 pad PB9: Net-(A1-PadPB9) -> PB9
- JP5 pad 1: Net-(A1-PadPB9) -> PB6
- JP5 pad 2: out3 -> out0
- JP6 pad 1: Net-(A1-PadPB8) -> PB7
- JP6 pad 2: out2 -> out1
- JP7 pad 1: Net-(A1-PadPB7) -> PB8
- JP7 pad 2: out1 -> out2
- JP8 pad 1: Net-(A1-PadPB6) -> PB9
- JP8 pad 2: out0 -> out3
- JP9 pad 1: +5V -> VCC
- R108 pad 1: Net-(D102-Pad1) -> Net-(D103-Pad1)
- R111 pad 1: Net-(D103-Pad1) -> Net-(D102-Pad1)
- U1 pad 12: Net-(JP13-Pad1) -> Net-(JP5-Pad3)
- U1 pad 13: Net-(JP12-Pad1) -> Net-(JP6-Pad3)
- U1 pad 14: Net-(JP11-Pad1) -> Net-(JP7-Pad3)
- U1 pad 15: Net-(JP10-Pad1) -> Net-(JP8-Pad3)
- U1 pad 5: Net-(A1-PadPB9) -> PB9
- U1 pad 6: Net-(A1-PadPB8) -> PB8
- U1 pad 7: Net-(A1-PadPB7) -> PB7
- U1 pad 8: Net-(A1-PadPB6) -> PB6
Routing:
- net VCC: track 0.00 -> 318.1 mm, vias 0 -> 6
- net GND: track 0.00 -> 252.1 mm, vias 0 -> 4
- net Net-(A1-PadPB14): track 0.00 -> 118.0 mm, vias 0 -> 3
- net MISO_MIDI: track 0.00 -> 110.1 mm, vias 0 -> 1
- net SCK_MIDI_5: track 0.00 -> 104.7 mm, vias 0 -> 4
- net in0: track 0.00 -> 103.1 mm, vias 0 -> 4
- net STROBE_MIDI_5: track 0.00 -> 102.3 mm, vias 0 -> 3
- net out0: track 0.00 -> 87.3 mm, vias 0 -> 3
- net out3: track 0.00 -> 80.6 mm, vias 0 -> 3
- net out2: track 0.00 -> 79.0 mm, vias 0 -> 2
- net MOSI_MIDI_5: track 0.00 -> 75.7 mm
- net Net-(A1-PadPB13): track 0.00 -> 73.8 mm, vias 0 -> 3
- net Net-(A1-PadPB15): track 0.00 -> 67.1 mm, vias 0 -> 3
- net in3: track 0.00 -> 58.6 mm, vias 0 -> 1
- net in1: track 0.00 -> 57.9 mm, vias 0 -> 2
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
Commit message: Re-order parts on din5_pcb
Parts:
- added G***: LOGO, windfisch:windfisch_smaller, F.Cu at (30.0, 109.5)
- added REF**: OSHW-Logo2_9.8x8mm_SilkScreen, Symbol:OSHW-Logo2_9.8x8mm_SilkScreen, F.Cu at (53.5, 110.5)
- added REF**: MountingHole_3.2mm_M3_DIN965, MountingHole:MountingHole_3.2mm_M3_DIN965, F.Cu at (64.5, 110.0)
- added REF**: MountingHole_3.2mm_M3_DIN965, MountingHole:MountingHole_3.2mm_M3_DIN965, F.Cu at (19.5, 110.0)
- added REF**: MountingHole_3.2mm_M3_DIN965, MountingHole:MountingHole_3.2mm_M3_DIN965, F.Cu at (64.5, 10.0)
- added REF**: MountingHole_3.2mm_M3_DIN965, MountingHole:MountingHole_3.2mm_M3_DIN965, F.Cu at (19.5, 10.0)
- A1: footprint footprints:BLUEPILL -> footprints:BLUEPILL-blackpill
- D104: footprint LED_THT:LED_D3.0mm_Horizontal_O3.81mm_Z6.0mm -> LED_THT:LED_D3.0mm_Horizontal_O1.27mm_Z2.0mm
- J1: footprint Connector_PinHeader_2.54mm:PinHeader_1x03_P2.54mm_Vertical -> Connector_PinHeader_2.54mm:PinHeader_1x03_P2.54mm_Horizontal
- JP14: footprint Jumper:SolderJumper-3_P1.3mm_Bridged12_RoundedPad1.0x1.5mm -> Jumper:SolderJumper-3_P1.3mm_Open_RoundedPad1.0x1.5mm
- JP9: footprint Jumper:SolderJumper-3_P1.3mm_Bridged12_RoundedPad1.0x1.5mm -> Jumper:SolderJumper-3_P1.3mm_Open_RoundedPad1.0x1.5mm; moved to B.Cu
- moved J2 7.68 mm to (39.5, 111.0), turned to 90 degrees
- moved J3 7.46 mm to (44.5, 9.00)
- moved A1 7.25 mm to (42.0, 31.8)
- moved JP14 7.25 mm to (32.0, 53.2)
- moved JP5 7.25 mm to (42.0, 48.8)
- moved JP6 7.25 mm to (42.0, 46.2)
- moved JP7 7.25 mm to (42.0, 43.8)
- moved JP8 7.25 mm to (42.0, 41.2)
- moved U1 7.25 mm to (38.0, 28.8)
- moved JP9 7.00 mm to (43.5, 30.0)
- moved J1 2.50 mm to (39.5, 16.0)
- moved U101 0.82 mm to (32.5, 68.1)
- moved C101 0.61 mm to (37.9, 71.9)
- moved R1 0.56 mm to (48.4, 98.5)
- moved U2 0.56 mm to (32.5, 83.3)
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Routing:
- net VCC: track 318.1 -> 0.00 mm, vias 6 -> 0
- net GND: track 252.1 -> 0.00 mm, vias 4 -> 0
- net Net-(A1-PadPB14): track 118.0 -> 0.00 mm, vias 3 -> 0
- net MISO_MIDI: track 110.1 -> 0.00 mm, vias 1 -> 0
- net SCK_MIDI_5: track 104.7 -> 0.00 mm, vias 4 -> 0
- net in0: track 103.1 -> 0.00 mm, vias 4 -> 0
- net STROBE_MIDI_5: track 102.3 -> 0.00 mm, vias 3 -> 0
- net out0: track 87.3 -> 0.00 mm, vias 3 -> 0
- net out3: track 80.6 -> 0.00 mm, vias 3 -> 0
- net out2: track 79.0 -> 0.00 mm, vias 2 -> 0
- net MOSI_MIDI_5: track 75.7 -> 0.00 mm
- net Net-(A1-PadPB13): track 73.8 -> 0.00 mm, vias 3 -> 0
- net Net-(A1-PadPB15): track 67.1 -> 0.00 mm, vias 3 -> 0
- net in3: track 58.6 -> 0.00 mm, vias 1 -> 0
- net in1: track 57.9 -> 0.00 mm, vias 2 -> 0
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Other:
- board outline added: 56 x 110 mm
- board text added: "245"
- board text added: "3.3V"
- board text added: "541"
- board text added: "5V"
- board text added: "from master"
- board text added: "midikraken (din5 rev01) (c) 2021 Florian Jung https://github.com/ Windfisch/midikraken"
- board text added: "pass thru"
- board text added: "to slave"

Commit message: intermediate commit
Other:
- outline, holes or cut-outs redrawn
Changed lines of the file:
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@@
   (general
     (thickness 1.6)
-    (drawings 28)
+    (drawings 32)
     (tracks 0)
     (zones 0)
@@
     )
   )
+  (gr_arc (start 46.5 5.75) (end 46.5 6.5) (angle -90) (layer Edge.Cuts) (width 0.05))
+  (gr_arc (start 48 5.75) (end 48 5) (angle -90) (layer Edge.Cuts) (width 0.05))
+  (gr_arc (start 37.5 5.75) (end 36.75 5.75) (angle -90) (layer Edge.Cuts) (width 0.05))
+  (gr_arc (start 36 5.75) (end 36.75 5.75) (angle -90) (layer Edge.Cuts) (width 0.05))
+  (gr_arc (start 46.5 114.25) (end 47.25 114.25) (angle -90) (layer Edge.Cuts) (width 0.05))
+  (gr_arc (start 48 114.25) (end 47.25 114.25) (angle -90) (layer Edge.Cuts) (width 0.05))
+  (gr_arc (start 37.5 114.25) (end 37.5 113.5) (angle -90) (layer Edge.Cuts) (width 0.05))
+  (gr_arc (start 36 114.25) (end 36 115) (angle -90) (layer Edge.Cuts) (width 0.05))
   (gr_line (start 14 9) (end 14 111) (layer Edge.Cuts) (width 0.05))
   (gr_line (start 36 5) (end 18 5) (layer Edge.Cuts) (width 0.05))
@@
   (gr_arc (start 18 111) (end 14 111) (angle -90) (layer Edge.Cuts) (width 0.05))
   (gr_arc (start 66 111) (end 66 115) (angle -90) (layer Edge.Cuts) (width 0.05))
-  (gr_line (start 46.5 113.5) (end 48 115) (layer Edge.Cuts) (width 0.05))
   (gr_line (start 37.5 113.5) (end 46.5 113.5) (layer Edge.Cuts) (width 0.05))
-  (gr_line (start 36 115) (end 37.5 113.5) (layer Edge.Cuts) (width 0.05))
-  (gr_line (start 46.5 6.5) (end 48 5) (layer Edge.Cuts) (width 0.05))
   (gr_line (start 37.5 6.5) (end 46.5 6.5) (layer Edge.Cuts) (width 0.05))
-  (gr_line (start 36 5) (end 37.5 6.5) (layer Edge.Cuts) (width 0.05))
   (gr_text "midikraken (din5 rev01)\n(c) 2021 Florian Jung\nhttps://github.com/\nWindfisch/midikraken" (at 42 62.5) (layer F.SilkS)
     (effects (font (size 1 1) (thickness 0.15)))

Commit message: Come layout considerations
Parts:
- removed the REF** at (53.5, 110.5)
- added REF**: PinHeader_2x02_P2.54mm_Vertical, Connector_PinHeader_2.54mm:PinHeader_2x02_P2.54mm_Vertical, F.Cu at (26.8, 6.90)
- added REF**: USB_A_Molex_105057_Vertical, Connector_USB:USB_A_Molex_105057_Vertical, F.Cu at (86.7, 15.4)
- added REF**: USB_Micro-B_Wuerth_629105150521, Connector_USB:USB_Micro-B_Wuerth_629105150521, F.Cu at (56.0, 9.90)
- added REF**: USB_Micro-B_Wuerth_629105150521, Connector_USB:USB_Micro-B_Wuerth_629105150521, F.Cu at (28.0, 9.90)
- added REF**: USB_A_Molex_105057_Vertical, Connector_USB:USB_A_Molex_105057_Vertical, B.Cu at (113.5, 31.0)
- added REF**: USB_A_Molex_105057_Vertical, Connector_USB:USB_A_Molex_105057_Vertical, B.Cu at (138.0, 32.7)
- added REF**: USB_A_Stewart_SS-52100-001_Horizontal, Connector_USB:USB_A_Stewart_SS-52100-001_Horizontal, F.Cu at (125.5, 61.0)
- added REF**: USB_A_Molex_67643_Horizontal, Connector_USB:USB_A_Molex_67643_Horizontal, F.Cu at (119.5, 55.5)
- added REF1: din5-frickel, footprints:din5-frickel, B.Cu at (65.2, 24.8)
- added REF2: din5-frickel, footprints:din5-frickel, B.Cu at (65.2, 50.0)
- added REF3: din5-frickel, footprints:din5-frickel, B.Cu at (65.2, 75.0)
- added REF4: din5-frickel, footprints:din5-frickel, B.Cu at (65.2, 100.0)
- added REF5: din5-frickel, footprints:din5-frickel, B.Cu at (18.8, 70.0)
- added REF51: din5-frickel, footprints:din5-frickel, B.Cu at (18.8, 95.2)
- added REF6: din5-frickel, footprints:din5-frickel, B.Cu at (18.8, 45.0)
- added REF7: din5-frickel, footprints:din5-frickel, B.Cu at (18.8, 20.0)
- added REFaa: RotaryEncoder_Alps_EC11E-Switch_Vertical_H20mm, Rotary_Encoder:RotaryEncoder_Alps_EC11E-Switch_Vertical_H20mm, B.Cu at (39.5, 68.3)
- added oh: OSHW-Logo2_9.8x8mm_SilkScreen, Symbol:OSHW-Logo2_9.8x8mm_SilkScreen, F.Cu at (55.0, 110.2)
- added refbb: PinHeader_1x07_P2.54mm_Vertical, Connector_PinHeader_2.54mm:PinHeader_1x07_P2.54mm_Vertical, B.Cu at (34.4, 65.0)
- moved R109 8.15 mm to (17.9, 86.0), turned to 180 degrees
- moved R110 7.91 mm to (66.1, 34.0), turned to 0 degrees
- moved R106 7.81 mm to (66.4, 84.0), turned to 0 degrees
- moved R105 7.73 mm to (17.9, 36.0), turned to 180 degrees
- moved JP5 7.25 mm to (42.0, 41.5)
- moved JP6 7.25 mm to (42.0, 39.0)
- moved JP7 7.25 mm to (42.0, 36.5)
- moved JP8 7.25 mm to (42.0, 34.0)
- moved JP9 7.25 mm to (43.5, 22.8)
- moved U1 7.25 mm to (38.0, 21.5)
- moved R209 5.65 mm to (28.5, 56.0), turned to 270 degrees
- moved R205 5.33 mm to (28.5, 39.1), turned to 90 degrees
- moved R102 5.19 mm to (28.5, 80.9), turned to 90 degrees
- moved R112 5.15 mm to (66.1, 36.0), turned to 0 degrees
- moved R111 5.14 mm to (17.9, 84.0), turned to 180 degrees
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- renumbered REF** to hole1, REF** to hole2, REF** to hole3, REF** to hole4, G*** to wf
Other:
- board text added: "midikraken (din rev01) (c) 2021 Florian Jung https://github.com/ Windfisch/midikraken"
- board text removed: "midikraken (din5 rev01) (c) 2021 Florian Jung https://github.com/ Windfisch/midikraken"

Commit message: intermediate commit
Parts:
- removed the REF** at (26.8, 6.90)
- removed the REF** at (56.0, 9.90)
- removed the REF** at (28.0, 9.90)
- removed REF1, REF2, REF6, REF7: din5-frickel, footprints:din5-frickel
- added J111: din5-frickel, footprints:din5-frickel, B.Cu at (18.8, 20.0)
- added J114: din5-frickel, footprints:din5-frickel, B.Cu at (65.2, 50.0)
- added J211: din5-frickel, footprints:din5-frickel, B.Cu at (18.8, 45.0)
- added J214: din5-frickel, footprints:din5-frickel, B.Cu at (65.2, 24.8)
- added J4: USB_Micro-B_Wuerth_629105150521, Connector_USB:USB_Micro-B_Wuerth_629105150521, F.Cu at (28.0, 10.1)
- added J5: USB_Micro-B_Wuerth_629105150521, Connector_USB:USB_Micro-B_Wuerth_629105150521, F.Cu at (56.0, 10.1)
- added J6: PinHeader_2x02_P2.54mm_Vertical, Connector_PinHeader_2.54mm:PinHeader_2x02_P2.54mm_Vertical, F.Cu at (26.7, 7.56)
- renumbered REF5 to J112, REF4 to J113, REF51 to J212, REF3 to J213
Other:
- outline, holes or cut-outs redrawn
Changed lines of the file:
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@@
   (general
     (thickness 1.6)
-    (drawings 32)
+    (drawings 34)
     (tracks 0)
     (zones 0)
@@
   )
   (module Connector_PinHeader_2.54mm:PinHeader_2x02_P2.54mm_Vertical (layer F.Cu)
-    (at 26.8 6.9)
+    (at 26.7 7.56)
     (descr "Through hole straight pin header, 2x02, 2.54mm pitch, double rows")
     (tags "Through hole pin header THT 2x02 2.54mm double row")
-    (fp_text reference REF** (at 1.27 -2.33) (layer F.SilkS)
+    (fp_text reference J6 (at 1.27 -2.33) (layer F.SilkS)
       (effects (font (size 1 1) (thickness 0.15)))
     )
@@
   )
   (module Connector_USB:USB_Micro-B_Wuerth_629105150521 (layer F.Cu)
-    (at 56 9.9 180)
+    (at 56 10.1 180)
     (descr "USB Micro-B receptacle, http://www.mouser.com/ds/2/445/629105150521-469306.pdf")
     (tags "usb micro receptacle")
     (attr smd)
-    (fp_text reference REF** (at 0 -3.5) (layer F.SilkS)
+    (fp_text reference J5 (at 0 -3.5) (layer F.SilkS)
       (effects (font (size 1 1) (thickness 0.15)))
     )
@@
   )
   (module Connector_USB:USB_Micro-B_Wuerth_629105150521 (layer F.Cu)
-    (at 28 9.9 180)
+    (at 28 10.1 180)
     (descr "USB Micro-B receptacle, http://www.mouser.com/ds/2/445/629105150521-469306.pdf")
     (tags "usb micro receptacle")
     (attr smd)
-    (fp_text reference REF** (at 0 -3.5) (layer F.SilkS)
+    (fp_text reference J4 (at 0 -3.5) (layer F.SilkS)
       (effects (font (size 1 1) (thickness 0.15)))
     )
@@
   (module footprints:din5-frickel (layer B.Cu)
     (at 18.75 95.25 225)
-    (fp_text reference REF51 (at 0 -6.604 225) (layer B.SilkS)
+    (fp_text reference J212 (at 0 -6.604 225) (layer B.SilkS)
       (effects (font (size 1 1) (thickness 0.15)) (justify mirror))
     )
@@
   (module footprints:din5-frickel (layer B.Cu)
     (at 18.75 45 225)
-    (fp_text reference REF6 (at 0 -6.604 225) (layer B.SilkS)
+    (fp_text reference J211 (at 0 -6.604 225) (layer B.SilkS)
       (effects (font (size 1 1) (thickness 0.15)) (justify mirror))
     )
@@
   (module footprints:din5-frickel (layer B.Cu)
     (at 18.75 70 225)
-    (fp_text reference REF5 (at 0 -6.604 225) (layer B.SilkS)
+    (fp_text reference J112 (at 3.853732 -5.76292 225) (layer B.SilkS)
       (effects (font (size 1 1) (thickness 0.15)) (justify mirror))
     )
@@
   (module footprints:din5-frickel (layer B.Cu)
     (at 18.75 20 225)
-    (fp_text reference REF7 (at 0 -6.604 225) (layer B.SilkS)
+    (fp_text reference J111 (at 4.419417 -6.045763 225) (layer B.SilkS)
       (effects (font (size 1 1) (thickness 0.15)) (justify mirror))
     )
@@
   (module footprints:din5-frickel (layer B.Cu)
     (at 65.25 100 45)
-    (fp_text reference REF4 (at 0 -6.604 225) (layer B.SilkS)
+    (fp_text reference J113 (at 0 -6.604 225) (layer B.SilkS)
       (effects (font (size 1 1) (thickness 0.15)) (justify mirror))
     )
@@
   (module footprints:din5-frickel (layer B.Cu)
     (at 65.25 75 45)
-    (fp_text reference REF3 (at 0 -6.604 225) (layer B.SilkS)
+    (fp_text reference J213 (at 0 -6.604 225) (layer B.SilkS)
       (effects (font (size 1 1) (thickness 0.15)) (justify mirror))
     )
@@
   (module footprints:din5-frickel (layer B.Cu)
     (at 65.25 50 45)
-    (fp_text reference REF2 (at 0 -6.604 225) (layer B.SilkS)
+    (fp_text reference J114 (at -5.126524 -2.863782 225) (layer B.SilkS)
       (effects (font (size 1 1) (thickness 0.15)) (justify mirror))
     )
@@
   (module footprints:din5-frickel (layer B.Cu)
     (at 65.25 24.75 45)
-    (fp_text reference REF1 (at 0 -6.604 225) (layer B.SilkS)
+    (fp_text reference J214 (at -5.091169 -2.899138 225) (layer B.SilkS)
       (effects (font (size 1 1) (thickness 0.15)) (justify mirror))
     )
@@
     )
   )
-  (gr_arc (start 46.5 5.75) (end 46.5 6.5) (angle -90) (layer Edge.Cuts) (width 0.05))
-  (gr_arc (start 48 5.75) (end 48 5) (angle -90) (layer Edge.Cuts) (width 0.05))
-  (gr_arc (start 37.5 5.75) (end 36.75 5.75) (angle -90) (layer Edge.Cuts) (width 0.05))
-  (gr_arc (start 36 5.75) (end 36.75 5.75) (angle -90) (layer Edge.Cuts) (width 0.05))
+  (gr_line (start 62.5 5) (end 66 5) (layer Edge.Cuts) (width 0.05))
+  (gr_line (start 46.5 6.5) (end 61 6.5) (layer Edge.Cuts) (width 0.05))
+  (gr_line (start 23 6.5) (end 37.5 6.5) (layer Edge.Cuts) (width 0.05))
+  (gr_line (start 18 5) (end 21.5 5) (layer Edge.Cuts) (width 0.05))
+  (gr_arc (start 61 5.75) (end 61 6.5) (angle -90) (layer Edge.Cuts) (width 0.05))
+  (gr_arc (start 62.5 5.75) (end 62.5 5) (angle -90) (layer Edge.Cuts) (width 0.05))
+  (gr_arc (start 23 5.75) (end 22.25 5.75) (angle -90) (layer Edge.Cuts) (width 0.05))
+  (gr_arc (start 21.5 5.75) (end 22.25 5.75) (angle -90) (layer Edge.Cuts) (width 0.05))
   (gr_arc (start 46.5 114.25) (end 47.25 114.25) (angle -90) (layer Edge.Cuts) (width 0.05))
   (gr_arc (start 48 114.25) (end 47.25 114.25) (angle -90) (layer Edge.Cuts) (width 0.05))
@@
   (gr_arc (start 36 114.25) (end 36 115) (angle -90) (layer Edge.Cuts) (width 0.05))
   (gr_line (start 14 9) (end 14 111) (layer Edge.Cuts) (width 0.05))
-  (gr_line (start 36 5) (end 18 5) (layer Edge.Cuts) (width 0.05))
-  (gr_line (start 66 5) (end 48 5) (layer Edge.Cuts) (width 0.05))
   (gr_line (start 70 111) (end 70 9) (layer Edge.Cuts) (width 0.05))
   (gr_line (start 48 115) (end 66 115) (layer Edge.Cuts) (width 0.05))

Commit message: din 5 pin pcb finished. todo: autoroute
Parts:
- removed REF** (x3): USB_A_Molex_105057_Vertical, Connector_USB:USB_A_Molex_105057_Vertical
- removed REF**: USB_A_Stewart_SS-52100-001_Horizontal, Connector_USB:USB_A_Stewart_SS-52100-001_Horizontal
- removed REF**: USB_A_Molex_67643_Horizontal, Connector_USB:USB_A_Molex_67643_Horizontal
- removed refbb: PinHeader_1x07_P2.54mm_Vertical, Connector_PinHeader_2.54mm:PinHeader_1x07_P2.54mm_Vertical
- added J7: Conn_02x02_Odd_Even, Connector_PinHeader_2.54mm:PinHeader_2x02_P2.54mm_Vertical, F.Cu at (54.7, 7.50)
- added J8: Conn_01x07, Connector_PinHeader_2.54mm:PinHeader_1x07_P2.54mm_Vertical, B.Cu at (34.4, 64.9)
- J111, J112, J113, J114, J211, J212, J213, J214: value din5-frickel -> do not equip
- J2, J3: value 2x3 female -> Conn_02x03_Odd_Even
- J4, J5: value USB_Micro-B_Wuerth_629105150521 -> USB_B_Micro
- J6: value PinHeader_2x02_P2.54mm_Vertical -> Conn_02x02_Odd_Even
- SW1: renamed from REFaa; value RotaryEncoder_Alps_EC11E-Switch_Vertical_H20mm -> Rotary_Encoder_Switch
Connections:
- net Net-(A1-PadPB13) renamed PB13
- net Net-(A1-PadPB15) renamed PB15
- A1 pad PA1: (no net) -> PA1
- A1 pad PA11: (no net) -> USB_DM
- A1 pad PA12: (no net) -> USB_DP
- A1 pad PA2: (no net) -> PA2
- A1 pad PA8: (no net) -> USB_ID
- A1 pad PC15: (no net) -> PC15
- J111 pad 4: (no net) -> Net-(J101-Pad4)
- J111 pad 5: (no net) -> Net-(J101-Pad5)
- J112 pad 4: (no net) -> Net-(J102-Pad5)
- J112 pad 5: (no net) -> Net-(J102-Pad5)
- J113 pad 4: (no net) -> Net-(J103-Pad4)
- J113 pad 5: (no net) -> Net-(J103-Pad5)
- J114 pad 4: (no net) -> Net-(J104-Pad5)
- J114 pad 5: (no net) -> Net-(J104-Pad5)
- J2 pad 2: MIDI_MOSI_CHAIN -> MIDI_MISO_CHAIN
- J2 pad 3: SCK_MIDI_5 -> MIDI_MOSI_CHAIN
- J2 pad 4: GND -> STROBE_MIDI_5
- J2 pad 5: STROBE_MIDI_5 -> SCK_MIDI_5
- J2 pad 6: MIDI_MISO_CHAIN -> GND
- J211 pad 2: (no net) -> GND
- J211 pad 4: (no net) -> Net-(J201-Pad4)
- J211 pad 5: (no net) -> Net-(J201-Pad5)
- J212 pad 2: (no net) -> GND
- J212 pad 4: (no net) -> Net-(J202-Pad4)
- J212 pad 5: (no net) -> Net-(J202-Pad5)
- J213 pad 2: (no net) -> GND
- J213 pad 4: (no net) -> Net-(J203-Pad4)
- J213 pad 5: (no net) -> Net-(J203-Pad5)
- J214 pad 2: (no net) -> GND
- J214 pad 4: (no net) -> Net-(J204-Pad4)
- J214 pad 5: (no net) -> Net-(J204-Pad5)
- J3 pad 2: MOSI_MIDI_5 -> MISO_MIDI
- J3 pad 3: SCK_MIDI_5 -> MOSI_MIDI_5
- J3 pad 4: GND -> STROBE_MIDI_5
- J3 pad 5: STROBE_MIDI_5 -> SCK_MIDI_5
- J3 pad 6: MISO_MIDI -> GND
- J4 pad 1: (no net) -> VCC
- J4 pad 2: (no net) -> USB_DM
- J4 pad 3: (no net) -> USB_DP
- J4 pad 4: (no net) -> USB_ID
- J4 pad 5: (no net) -> GND
- J4 pad 6: (no net) -> Net-(J4-Pad6)
- J5 pad 1: (no net) -> VCC
- J5 pad 5: (no net) -> GND
- J5 pad 6: (no net) -> Net-(J5-Pad6)
- J6 pad 1: (no net) -> VCC
- J6 pad 2: (no net) -> USB_DP
- J6 pad 3: (no net) -> GND
- J6 pad 4: (no net) -> USB_DM
- SW1 pad A: (no net) -> PB6
- SW1 pad B: (no net) -> PB7
- SW1 pad C: (no net) -> GND
- SW1 pad S1: (no net) -> PC15
- SW1 pad S2: (no net) -> GND

Commit message: Autorouted board, added 3d models
Parts:
- moved C102 51.5 mm to (98.6, 91.6)
- moved J3 51.5 mm to (93.5, 25.0)
- moved R202 51.5 mm to (71.1, 104.5)
- moved A1 51.5 mm to (91.0, 47.8)
- moved D101 51.5 mm to (70.0, 49.8)
- moved D102 51.5 mm to (70.0, 99.5)
- moved D103 51.5 mm to (112.2, 102.2)
- moved D104 51.5 mm to (112.0, 52.2)
- moved D201 51.5 mm to (72.5, 49.8)
- moved D202 51.5 mm to (72.5, 99.5)
- moved D203 51.5 mm to (109.8, 102.2)
- moved D204 51.5 mm to (109.5, 52.2)
- moved J101 51.5 mm to (70.0, 38.5)
- moved J102 51.5 mm to (70.0, 88.5)
- moved J103 51.5 mm to (112.0, 113.5)
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Routing:
- net VCC: track 0.00 -> 408.6 mm, vias 0 -> 1
- net GND: track 0.00 -> 336.9 mm, vias 0 -> 4
- net MISO_MIDI: track 0.00 -> 167.6 mm, vias 0 -> 2
- net SCK_MIDI_5: track 0.00 -> 130.2 mm
- net Net-(A1-PadPB14): track 0.00 -> 110.5 mm, vias 0 -> 2
- net STROBE_MIDI_5: track 0.00 -> 106.4 mm, vias 0 -> 1
- net MOSI_MIDI_5: track 0.00 -> 103.7 mm, vias 0 -> 2
- net out0: track 0.00 -> 102.5 mm, vias 0 -> 1
- net in0: track 0.00 -> 96.2 mm, vias 0 -> 1
- net out2: track 0.00 -> 94.9 mm, vias 0 -> 1
- net out3: track 0.00 -> 87.3 mm, vias 0 -> 1
- net in3: track 0.00 -> 82.2 mm
- net PB13: track 0.00 -> 81.3 mm, vias 0 -> 1
- net PB15: track 0.00 -> 75.1 mm, vias 0 -> 1
- net Net-(J101-Pad5): track 0.00 -> 73.9 mm
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- added copper zone on B.Cu, net GND
- added copper zone on F.Cu, net GND
