File: schem/din5_pcb/din5_pcb.kicad_pcb (KiCad board)
At the start: 2 copper layers, 56 x 110 mm, 82 parts, among them J1 Conn_01x03_Male, J101 DIN-5_180degree, J102 DIN-5_180degree, J103 DIN-5_180degree, J104 DIN-5_180degree, J111 do not equip, J112 do not equip, J113 do not equip, J114 do not equip, J2 Conn_02x03_Odd_Even, J201 DIN-5_180degree, J202 DIN-5_180degree, J203 DIN-5_180degree, J204 DIN-5_180degree, J211 do not equip, J212 do not equip, J213 do not equip, J214 do not equip, J3 Conn_02x03_Odd_Even, J4 USB_B_Micro, J5 USB_B_Micro, J6 Conn_02x02_Odd_Even, J7 Conn_02x02_Odd_Even, J8 Conn_01x07, SW1 Rotary_Encoder_Switch, U1 74HCT245, U101 HCPL-2630, U102 HCPL-2630, U2 74HC595, U3 74HC165

Commit message: final commit[tm] for the din 5 pcb
Other:
- board text added: "Power only!"
- board text added: "USB host only!"
Changed lines of the file:
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@@
   (general
     (thickness 1.6)
-    (drawings 34)
+    (drawings 36)
     (tracks 1049)
     (zones 0)
@@
     (descr "Through hole straight pin header, 2x02, 2.54mm pitch, double rows")
     (tags "Through hole pin header THT 2x02 2.54mm double row")
-    (fp_text reference J7 (at 1.27 -2.33) (layer F.SilkS)
+    (fp_text reference J7 (at -2.45 2.5) (layer F.SilkS)
       (effects (font (size 1 1) (thickness 0.15)))
     )
@@
     (pad 1 thru_hole rect (at 0 0) (size 1.7 1.7) (drill 1) (layers *.Cu *.Mask)
       (net 12 VCC))
-    (model ${KISYS3DMOD}/Connector_PinHeader_2.54mm.3dshapes/PinHeader_2x02_P2.54mm_Vertical.wrl
-      (at (xyz 0 0 0))
-      (scale (xyz 1 1 1))
-      (rotate (xyz 0 0 0))
-    )
   )
   (module Connector_PinHeader_2.54mm:PinHeader_2x02_P2.54mm_Vertical (layer F.Cu)
@@
     (descr "Through hole straight pin header, 2x02, 2.54mm pitch, double rows")
     (tags "Through hole pin header THT 2x02 2.54mm double row")
-    (fp_text reference J6 (at 1.27 -2.33) (layer F.SilkS)
+    (fp_text reference J6 (at -2.7 2.44) (layer F.SilkS)
       (effects (font (size 1 1) (thickness 0.15)))
     )
@@
     (pad 1 thru_hole rect (at 0 0) (size 1.7 1.7) (drill 1) (layers *.Cu *.Mask)
       (net 12 VCC))
-    (model ${KISYS3DMOD}/Connector_PinHeader_2.54mm.3dshapes/PinHeader_2x02_P2.54mm_Vertical.wrl
-      (at (xyz 0 0 0))
-      (scale (xyz 1 1 1))
-      (rotate (xyz 0 0 0))
-    )
   )
   (module Connector_PinHeader_2.54mm:PinHeader_2x03_P2.54mm_Vertical (layer F.Cu)
@@
     (tags "usb micro receptacle")
     (attr smd)
-    (fp_text reference J5 (at 0 -3.5) (layer F.SilkS)
+    (fp_text reference J5 (at 4 -4.15) (layer F.SilkS)
       (effects (font (size 1 1) (thickness 0.15)))
     )
@@
     (pad "" np_thru_hole oval (at -2.5 -0.8 180) (size 0.8 0.8) (drill 0.8) (layers *.Cu *.Mask))
     (pad "" np_thru_hole oval (at 2.5 -0.8 180) (size 0.8 0.8) (drill 0.8) (layers *.Cu *.Mask))
-    (model ${KISYS3DMOD}/Connector_USB.3dshapes/USB_Micro-B_Wuerth_629105150521.wrl
-      (at (xyz 0 0 0))
+    (model ../lib/3d/microUSB-B.STEP
+      (offset (xyz 0 -3.5 1.5))
       (scale (xyz 1 1 1))
-      (rotate (xyz 0 0 0))
+      (rotate (xyz -90 0 180))
     )
   )
@@
     (tags "usb micro receptacle")
     (attr smd)
-    (fp_text reference J4 (at 0 -3.5) (layer F.SilkS)
+    (fp_text reference J4 (at -2.75 -4.15) (layer F.SilkS)
       (effects (font (size 1 1) (thickness 0.15)))
     )
@@
     (pad 1 smd rect (at -1.3 -1.9 180) (size 0.45 1.3) (layers F.Cu F.Paste F.Mask)
       (net 12 VCC))
-    (model ${KISYS3DMOD}/Connector_USB.3dshapes/USB_Micro-B_Wuerth_629105150521.wrl
-      (at (xyz 0 0 0))
+    (model ../lib/3d/microUSB-B.STEP
+      (offset (xyz 0 -3.5 1.5))
       (scale (xyz 1 1 1))
-      (rotate (xyz 0 0 0))
+      (rotate (xyz -90 0 180))
     )
   )
@@
     )
   )
+  (gr_text "Power\nonly!" (at 112.25 27.75) (layer F.SilkS)
+    (effects (font (size 1 1) (thickness 0.15)))
+  )
+  (gr_text "USB host\nonly!" (at 72 27.75) (layer F.SilkS)
+    (effects (font (size 1 1) (thickness 0.15)) (justify right))
+  )
   (gr_line (start 111.5 21) (end 115 21) (layer Edge.Cuts) (width 0.05))
