File: schem/din5_pcb/din5_pcb.kicad_pcb (KiCad board)
At the start: 2 copper layers, 56 x 110 mm, 82 parts, among them J1 Conn_01x03_Male, J101 DIN-5_180degree, J102 DIN-5_180degree, J103 DIN-5_180degree, J104 DIN-5_180degree, J111 do not equip, J112 do not equip, J113 do not equip, J114 do not equip, J2 Conn_02x03_Odd_Even, J201 DIN-5_180degree, J202 DIN-5_180degree, J203 DIN-5_180degree, J204 DIN-5_180degree, J211 do not equip, J212 do not equip, J213 do not equip, J214 do not equip, J3 Conn_02x03_Odd_Even, J4 USB_B_Micro, J5 USB_B_Micro, J6 Conn_02x02_Odd_Even, J7 Conn_02x02_Odd_Even, J8 Conn_01x07, SW1 Rotary_Encoder_Switch, U1 74HCT245, U101 HCPL-2630, U102 HCPL-2630, U2 74HC595, U3 74HC165

Commit message: Increase bluepill hole size and reroute
Connections:
- J112 pad 4: Net-(J102-Pad5) -> Net-(J102-Pad4)
- J114 pad 4: Net-(J104-Pad5) -> Net-(J104-Pad4)
Routing:
- net GND: track 336.9 -> 0.00 mm, vias 4 -> 0
- net VCC: track 408.6 -> 328.3 mm
- net out3: track 87.3 -> 151.8 mm, vias 1 -> 0
- net MISO_MIDI: track 167.6 -> 124.1 mm, vias 2 -> 1
- net in1: track 63.2 -> 101.6 mm
- net Net-(A1-PadPC14): track 48.0 -> 27.3 mm, vias 0 -> 2
- net PB13: track 81.3 -> 101.7 mm
- net Net-(J104-Pad4): track 2.47 -> 15.5 mm
- net Net-(J102-Pad4): track 2.47 -> 15.5 mm
- net USB_DP: track 23.8 -> 36.8 mm
- net PB15: track 75.1 -> 84.1 mm
- net PB6: track 38.5 -> 47.0 mm
- net in3: track 82.2 -> 74.0 mm
- net SCK_MIDI_5: track 130.2 -> 122.6 mm, vias 0 -> 2
- net MOSI_MIDI_5: track 103.7 -> 96.5 mm, vias 2 -> 1
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
Commit message: reroute one track
Routing:
- net out3: track 151.8 -> 118.2 mm, vias 0 -> 1
- net GND: track 0.00 -> 31.4 mm
Changed lines of the file:
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@@
     (thickness 1.6)
     (drawings 36)
-    (tracks 899)
+    (tracks 906)
     (zones 0)
     (modules 82)
@@
   (segment (start 81 67.95) (end 82.23 67.95) (width 0.25) (layer B.Cu) (net 1))
   (segment (start 82.23 67.95) (end 83.38 66.8) (width 0.25) (layer B.Cu) (net 1))
+  (segment (start 117.566517 115.910481) (end 117.566517 112.066517) (width 0.25) (layer F.Cu) (net 2))
+  (segment (start 109.016998 124.46) (end 117.566517 115.910481) (width 0.25) (layer F.Cu) (net 2))
+  (segment (start 93.54 124.46) (end 109.016998 124.46) (width 0.25) (layer F.Cu) (net 2))
   (segment (start 81.7575 42.7066) (end 81.7575 36.2022) (width 0.25) (layer B.Cu) (net 3))
   (segment (start 81.7575 36.2022) (end 82.9097 35.05) (width 0.25) (layer B.Cu) (net 3))
@@
   (segment (start 96.8882 47.825) (end 104.5 47.825) (width 0.25) (layer B.Cu) (net 24))
   (segment (start 91 50) (end 91 48.9247) (width 0.25) (layer B.Cu) (net 24))
-  (segment (start 109.5 53.9083) (end 109.5 52.25) (width 0.25) (layer F.Cu) (net 24))
-  (segment (start 117.698409 62.106709) (end 109.5 53.9083) (width 0.25) (layer F.Cu) (net 24))
-  (segment (start 117.698409 65.778589) (end 117.698409 62.106709) (width 0.25) (layer F.Cu) (net 24))
-  (segment (start 115.604999 67.871999) (end 117.698409 65.778589) (width 0.25) (layer F.Cu) (net 24))
-  (segment (start 115.604999 87.225632) (end 115.604999 67.871999) (width 0.25) (layer F.Cu) (net 24))
-  (segment (start 81.475 106.39) (end 81.475 107.5153) (width 0.25) (layer F.Cu) (net 24))
-  (segment (start 81.475 107.5153) (end 81.7564 107.5153) (width 0.25) (layer F.Cu) (net 24))
-  (segment (start 117.566517 90.910481) (end 117.566517 89.18715) (width 0.25) (layer F.Cu) (net 24))
-  (segment (start 81.7564 107.5153) (end 82.6003 108.3592) (width 0.25) (layer F.Cu) (net 24))
-  (segment (start 82.6003 108.3592) (end 82.6003 123.3409) (width 0.25) (layer F.Cu) (net 24))
-  (segment (start 117.60065 115.10065) (end 117.60065 114.221283) (width 0.25) (layer F.Cu) (net 24))
-  (segment (start 87.4772 128.2178) (end 104.4835 128.2178) (width 0.25) (layer F.Cu) (net 24))
-  (segment (start 104.4835 128.2178) (end 117.60065 115.10065) (width 0.25) (layer F.Cu) (net 24))
-  (segment (start 82.6003 123.3409) (end 87.4772 128.2178) (width 0.25) (layer F.Cu) (net 24))
-  (segment (start 115.604999 112.225632) (end 115.604999 92.871999) (width 0.25) (layer F.Cu) (net 24))
-  (segment (start 117.60065 114.221283) (end 115.604999 112.225632) (width 0.25) (layer F.Cu) (net 24))
-  (segment (start 115.604999 92.871999) (end 117.566517 90.910481) (width 0.25) (layer F.Cu) (net 24))
-  (segment (start 117.566517 89.18715) (end 115.604999 87.225632) (width 0.25) (layer F.Cu) (net 24))
+  (via (at 103 106.5) (size 0.8) (drill 0.4) (layers F.Cu B.Cu) (net 24))
+  (segment (start 101.984999 107.515001) (end 103 106.5) (width 0.25) (layer B.Cu) (net 24))
+  (segment (start 99.984999 107.515001) (end 101.984999 107.515001) (width 0.25) (layer B.Cu) (net 24))
+  (segment (start 97.444999 110.055001) (end 99.984999 107.515001) (width 0.25) (layer B.Cu) (net 24))
+  (segment (start 85.140001 110.055001) (end 97.444999 110.055001) (width 0.25) (layer B.Cu) (net 24))
+  (segment (start 81.475 106.39) (end 85.140001 110.055001) (width 0.25) (layer B.Cu) (net 24))
+  (segment (start 109.5 53.4) (end 109.5 52.25) (width 0.25) (layer F.Cu) (net 24))
+  (segment (start 117.698402 61.598402) (end 109.5 53.4) (width 0.25) (layer F.Cu) (net 24))
+  (segment (start 117.566517 90.08766) (end 117.566517 86.089519) (width 0.25) (layer F.Cu) (net 24))
+  (segment (start 113.475001 94.179176) (end 117.566517 90.08766) (width 0.25) (layer F.Cu) (net 24))
+  (segment (start 113.475001 103.410001) (end 113.475001 94.179176) (width 0.25) (layer F.Cu) (net 24))
+  (segment (start 117.698402 65.593308) (end 117.698402 61.598402) (width 0.25) (layer F.Cu) (net 24))
+  (segment (start 113.410001 103.475001) (end 113.475001 103.410001) (width 0.25) (layer F.Cu) (net 24))
+  (segment (start 111.466125 103.475001) (end 113.410001 103.475001) (width 0.25) (layer F.Cu) (net 24))
+  (segment (start 106.584128 108.356998) (end 111.466125 103.475001) (width 0.25) (layer F.Cu) (net 24))
+  (segment (start 106.5 108.356998) (end 106.584128 108.356998) (width 0.25) (layer F.Cu) (net 24))
+  (segment (start 104.643002 106.5) (end 106.5 108.356998) (width 0.25) (layer F.Cu) (net 24))
+  (segment (start 103 106.5) (end 104.643002 106.5) (width 0.25) (layer F.Cu) (net 24))
+  (segment (start 115.395855 83.918857) (end 115.488499 84.011501) (width 0.25) (layer F.Cu) (net 24))
+  (segment (start 117.566517 86.089519) (end 115.488499 84.011501) (width 0.25) (layer F.Cu) (net 24))
+  (segment (start 115.395855 67.895855) (end 115.395855 83.918857) (width 0.25) (layer F.Cu) (net 24))
+  (segment (start 115.395855 67.895855) (end 117.698402 65.593308) (width 0.25) (layer F.Cu) (net 24))
   (segment (start 98.2625 116.55) (end 92.27 122.5425) (width 0.25) (layer B.Cu) (net 25))
   (segment (start 92.27 122.5425) (end 92.27 124.8548) (width 0.25) (layer B.Cu) (net 25))

Commit message: move connectors inwards, reroute
Parts:
- J2, J3: footprint Connector_PinHeader_2.54mm:PinHeader_2x03_P2.54mm_Vertical -> Connector_IDC:IDC-Header_2x03_P2.54mm_Vertical
- moved J8 4.90 mm to (83.4, 76.0)
- moved J2 1.00 mm to (88.5, 126.0)
- moved J3 1.00 mm to (93.5, 26.0)
- moved SW1 1.00 mm to (88.5, 83.3)
- moved U2 1.00 mm to (81.5, 100.3)
- moved U3 1.00 mm to (92.9, 100.3)
Connections:
- J8 pad 2: +5V -> +3V3
Routing:
- net GND: track 31.4 -> 330.5 mm
- net VCC: track 328.3 -> 366.0 mm, vias 1 -> 2
- net out3: track 118.2 -> 84.6 mm
- net PB13: track 101.7 -> 81.5 mm
- net +5V: track 18.0 -> 2.86 mm
- net out0: track 100.1 -> 87.9 mm, vias 0 -> 1
- net Net-(A1-PadPB12): track 24.0 -> 35.8 mm
- net MISO_MIDI: track 124.1 -> 133.6 mm, vias 1 -> 0
- net PB6: track 47.0 -> 38.0 mm, vias 1 -> 0
- net SCK_MIDI_5: track 122.6 -> 113.7 mm, vias 2 -> 0
- net STROBE_MIDI_5: track 109.3 -> 118.2 mm, vias 1 -> 0
- net USB_DP: track 36.8 -> 28.1 mm
- net in1: track 101.6 -> 93.9 mm
- net PA1: track 23.8 -> 18.9 mm
- net in0: track 90.9 -> 95.8 mm, vias 0 -> 1
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Other:
- board text added: "1"
- board text added: "2"

Commit message: Fix silkscreen, final touches
Parts:
- moved wf 2.04 mm to (76.5, 125.0), turned to 345 degrees
- moved oh 0.46 mm to (104.5, 126.2)
Routing:
- net GND: track 330.5 -> 401.3 mm, vias 0 -> 5
Other:
- board text added: "G"
- board text added: "JLCJLCJLCJLC"
- board text added: "d+"
- board text added: "d-"
