File: schem/din5_pcb/din5_pcb.sch (KiCad schematic (older format))
At the start: 74 parts, among them J1 Conn_01x03_Male, J101 DIN-5_180degree, J102 DIN-5_180degree, J103 DIN-5_180degree, J104 DIN-5_180degree, J111 do not equip, J112 do not equip, J113 do not equip, J114 do not equip, J2 2x3 female, J201 DIN-5_180degree, J202 DIN-5_180degree, J203 DIN-5_180degree, J204 DIN-5_180degree, J211 do not equip, J212 do not equip, J213 do not equip, J214 do not equip, J3 2x3 female, J4 USB_B_Micro, J5 USB_B_Micro, J6 Conn_02x02_Counter_Clockwise, J7 Conn_02x02_Counter_Clockwise, U1 74HCT245, U101 HCPL-2630, U102 HCPL-2630, U2 74HC595, U3 74HC165

Commit message: intermediate commit
Parts:
- removed J2, J3: 2x3 female, Connector_PinHeader_2.54mm:PinHeader_2x03_P2.54mm_Vertical, symbol Connector_Generic:Conn_02x03_Counter_Clockwise
- removed J6, J7: Conn_02x02_Counter_Clockwise, symbol Connector_Generic:Conn_02x02_Counter_Clockwise
- added J2, J3: Conn_02x03_Odd_Even, Connector_PinSocket_2.54mm:PinSocket_2x03_P2.54mm_Vertical, symbol Connector_Generic:Conn_02x03_Odd_Even
- added J6, J7: Conn_02x02_Odd_Even, Connector_PinSocket_2.54mm:PinSocket_2x02_P2.54mm_Vertical, symbol Connector_Generic:Conn_02x02_Odd_Even
- J111, J112, J113, J114, J211, J212, J213, J214: footprint footprints:DIN5 -> footprints:din5-frickel
- J4, J5: footprint (none) -> Connector_USB:USB_Micro-B_Wuerth_629105150521
Connections:
- net GND: now also J2.5 (Pin_5), J3.5 (Pin_5), J6.4 (Pin_4), J7.1 (Pin_1), J7.3 (Pin_3)
- net MIDI_MISO_CHAIN: now also J2.1 (Pin_1)
- net MIDI_MOSI_CHAIN: now also J2.4 (Pin_4)
- net MISO_MIDI: now also J3.1 (Pin_1)
- net MOSI_MIDI_5: now also J3.4 (Pin_4)
- net SCK_MIDI_5: now also J2.6 (Pin_6), J3.6 (Pin_6)
- net STROBE_MIDI_5: now also J2.3 (Pin_3), J3.3 (Pin_3)
- net USB_DM: now also J6.3 (Pin_3)
- net USB_DP: now also J6.1 (Pin_1)
- net VCC: now also J2.2 (Pin_2), J3.2 (Pin_2), J6.2 (Pin_2), J7.2 (Pin_2), J7.4 (Pin_4)
Other:
- note removed: "TODO: pinouts richtig drehen..."
Changed lines of the file:
@@
 F 0 "J211" H 6475 4150 50  0000 C CNN
 F 1 "do not equip" H 6525 3975 50  0000 C CNN
-F 2 "footprints:DIN5" H 6525 4225 50  0001 C CNN
+F 2 "footprints:din5-frickel" H 6525 4225 50  0001 C CNN
 F 3 "http://www.mouser.com/ds/2/18/40_c091_abd_e-75918.pdf" H 6525 4225 50  0001 C CNN
 	1    6525 4225
@@
 F 0 "J212" H 6475 5150 50  0000 C CNN
 F 1 "do not equip" H 6525 4975 50  0000 C CNN
-F 2 "footprints:DIN5" H 6525 5225 50  0001 C CNN
+F 2 "footprints:din5-frickel" H 6525 5225 50  0001 C CNN
 F 3 "http://www.mouser.com/ds/2/18/40_c091_abd_e-75918.pdf" H 6525 5225 50  0001 C CNN
 	1    6525 5225
@@
 F 0 "J213" H 6475 6150 50  0000 C CNN
 F 1 "do not equip" H 6525 5975 50  0000 C CNN
-F 2 "footprints:DIN5" H 6525 6225 50  0001 C CNN
+F 2 "footprints:din5-frickel" H 6525 6225 50  0001 C CNN
 F 3 "http://www.mouser.com/ds/2/18/40_c091_abd_e-75918.pdf" H 6525 6225 50  0001 C CNN
 	1    6525 6225
@@
 F 0 "J214" H 6475 7150 50  0000 C CNN
 F 1 "do not equip" H 6525 6975 50  0000 C CNN
-F 2 "footprints:DIN5" H 6525 7225 50  0001 C CNN
+F 2 "footprints:din5-frickel" H 6525 7225 50  0001 C CNN
 F 3 "http://www.mouser.com/ds/2/18/40_c091_abd_e-75918.pdf" H 6525 7225 50  0001 C CNN
 	1    6525 7225
@@
 	1    0    0    -1
 $EndComp
-$Comp
-L Connector_Generic:Conn_02x03_Counter_Clockwise J3
-U 1 1 60B5097F
-P 10000 6075
-F 0 "J3" H 10050 6350 50  0000 C CNN
-F 1 "2x3 female" H 9975 5850 50  0000 C CNN
-F 2 "Connector_PinHeader_2.54mm:PinHeader_2x03_P2.54mm_Vertical" H 10000 6075 50  0001 C CNN
-F 3 "~" H 10000 6075 50  0001 C CNN
-	1    10000 6075
-	1    0    0    -1
-$EndComp
 Text Notes 9625 5675 0    50   ~ 0
 chain to slave
@@
 F 3 "" H 10300 5450 50  0001 C CNN
 	1    10300 5450
-	1    0    0    -1
-$EndComp
-$Comp
-L Connector_Generic:Conn_02x03_Counter_Clockwise J2
-U 1 1 60B33612
-P 10000 5350
-F 0 "J2" H 10050 5625 50  0000 C CNN
-F 1 "2x3 female" H 9975 5125 50  0000 C CNN
-F 2 "Connector_PinHeader_2.54mm:PinHeader_2x03_P2.54mm_Vertical" H 10000 5350 50  0001 C CNN
-F 3 "~" H 10000 5350 50  0001 C CNN
-	1    10000 5350
 	1    0    0    -1
 $EndComp
@@
 F 0 "J5" H 7707 5567 50  0000 C CNN
 F 1 "USB_B_Micro" H 7707 5476 50  0000 C CNN
-F 2 "" H 7800 5050 50  0001 C CNN
+F 2 "Connector_USB:USB_Micro-B_Wuerth_629105150521" H 7800 5050 50  0001 C CNN
 F 3 "~" H 7800 5050 50  0001 C CNN
 	1    7650 5100
@@
 F 0 "J111" H 675 4375 50  0000 C CNN
 F 1 "do not equip" H 825 3900 50  0000 C CNN
-F 2 "footprints:DIN5" H 825 4150 50  0001 C CNN
+F 2 "footprints:din5-frickel" H 825 4150 50  0001 C CNN
 F 3 "http://www.mouser.com/ds/2/18/40_c091_abd_e-75918.pdf" H 825 4150 50  0001 C CNN
 	1    825  4150
@@
 F 0 "J113" H 675 6300 50  0000 C CNN
 F 1 "do not equip" H 825 5825 50  0000 C CNN
-F 2 "footprints:DIN5" H 825 6075 50  0001 C CNN
+F 2 "footprints:din5-frickel" H 825 6075 50  0001 C CNN
 F 3 "http://www.mouser.com/ds/2/18/40_c091_abd_e-75918.pdf" H 825 6075 50  0001 C CNN
 	1    825  6075
@@
 F 0 "J112" H 675 5225 50  0000 C CNN
 F 1 "do not equip" H 825 5475 50  0000 C CNN
-F 2 "footprints:DIN5" H 825 5000 50  0001 C CNN
+F 2 "footprints:din5-frickel" H 825 5000 50  0001 C CNN
 F 3 "http://www.mouser.com/ds/2/18/40_c091_abd_e-75918.pdf" H 825 5000 50  0001 C CNN
 	1    825  5000
@@
 F 0 "J114" H 675 7150 50  0000 C CNN
 F 1 "do not equip" H 825 7400 50  0000 C CNN
-F 2 "footprints:DIN5" H 825 6925 50  0001 C CNN
+F 2 "footprints:din5-frickel" H 825 6925 50  0001 C CNN
 F 3 "http://www.mouser.com/ds/2/18/40_c091_abd_e-75918.pdf" H 825 6925 50  0001 C CNN
 	1    825  6925
@@
 F 0 "J4" H 7707 4192 50  0000 C CNN
 F 1 "USB_B_Micro" H 7707 4101 50  0000 C CNN
-F 2 "" H 7800 3675 50  0001 C CNN
+F 2 "Connector_USB:USB_Micro-B_Wuerth_629105150521" H 7800 3675 50  0001 C CNN
 F 3 "~" H 7800 3675 50  0001 C CNN
 	1    7650 3725
@@
 	1    0    0    -1
 $EndComp
-$Comp
-L Connector_Generic:Conn_02x02_Counter_Clockwise J7
-U 1 1 60C35D31
-P 8600 3675
-F 0 "J7" H 8650 3800 50  0000 C CNN
-F 1 "Conn_02x02_Counter_Clockwise" H 8650 3801 50  0001 C CNN
-F 2 "" H 8600 3675 50  0001 C CNN
-F 3 "~" H 8600 3675 50  0001 C CNN
-	1    8600 3675
-	1    0    0    -1
-$EndComp
-$Comp
-L Connector_Generic:Conn_02x02_Counter_Clockwise J6
-U 1 1 60C41A1F
-P 8275 5200
-F 0 "J6" H 8325 5300 50  0000 C CNN
-F 1 "Conn_02x02_Counter_Clockwise" H 9300 5150 50  0001 C CNN
-F 2 "" H 8275 5200 50  0001 C CNN
-F 3 "~" H 8275 5200 50  0001 C CNN
-	1    8275 5200
-	1    0    0    -1
-$EndComp
 NoConn ~ 7950 5300
 $Comp
@@
 Wire Wire Line
 	8075 5200 8075 5300
-Connection ~ 8075 5200
 $Comp
 L power:GND #PWR0121
@@
 Wire Wire Line
 	8575 5200 8575 5300
-Connection ~ 8575 5300
 Text Notes 7900 5475 0    50   ~ 0
 power only!
@@
 Text Notes 8525 4000 0    50   ~ 0
 to eurorack USB-A\nsocket for host
-Text Notes 9775 3625 0    50   ~ 0
-TODO: pinouts richtig drehen...
+$Comp
+L Connector_Generic:Conn_02x03_Odd_Even J2
+U 1 1 60E04254
+P 10100 5350
+F 0 "J2" H 10150 5575 50  0000 C CNN
+F 1 "Conn_02x03_Odd_Even" H 10150 5576 50  0001 C CNN
+F 2 "Connector_PinSocket_2.54mm:PinSocket_2x03_P2.54mm_Vertical" H 10100 5350 50  0001 C CNN
+F 3 "~" H 10100 5350 50  0001 C CNN
+	1    10100 5350
+	-1   0    0    -1
+$EndComp
+$Comp
+L Connector_Generic:Conn_02x03_Odd_Even J3
+U 1 1 60E118D4
+P 10100 6075
+F 0 "J3" H 10150 6300 50  0000 C CNN
+F 1 "Conn_02x03_Odd_Even" H 10150 6301 50  0001 C CNN
+F 2 "Connector_PinSocket_2.54mm:PinSocket_2x03_P2.54mm_Vertical" H 10100 6075 50  0001 C CNN
+F 3 "~" H 10100 6075 50  0001 C CNN
+	1    10100 6075
+	-1   0    0    -1
+$EndComp
+$Comp
+L Connector_Generic:Conn_02x02_Odd_Even J7
+U 1 1 60E1FECA
+P 8375 5200
+F 0 "J7" H 8425 5325 50  0000 C CNN
+F 1 "Conn_02x02_Odd_Even" H 8425 5326 50  0001 C CNN
+F 2 "Connector_PinSocket_2.54mm:PinSocket_2x02_P2.54mm_Vertical" H 8375 5200 50  0001 C CNN
+F 3 "~" H 8375 5200 50  0001 C CNN
+	1    8375 5200
+	-1   0    0    -1
+$EndComp
+$Comp
+L Connector_Generic:Conn_02x02_Odd_Even J6
+U 1 1 60E2ACED
+P 8700 3675
+F 0 "J6" H 8750 3800 50  0000 C CNN
+F 1 "Conn_02x02_Odd_Even" H 8750 3801 50  0001 C CNN
+F 2 "Connector_PinSocket_2.54mm:PinSocket_2x02_P2.54mm_Vertical" H 8700 3675 50  0001 C CNN
+F 3 "~" H 8700 3675 50  0001 C CNN
+	1    8700 3675
+	-1   0    0    -1
+$EndComp
+Connection ~ 8075 5200
+Connection ~ 8575 5300
 $EndSCHEMATC
