File: schem/din5_pcb/din5_pcb.sch (KiCad schematic (older format))
At the start: 76 parts, among them J1 Conn_01x03_Male, J101 DIN-5_180degree, J102 DIN-5_180degree, J103 DIN-5_180degree, J104 DIN-5_180degree, J111 do not equip, J112 do not equip, J113 do not equip, J114 do not equip, J2 Conn_02x03_Odd_Even, J201 DIN-5_180degree, J202 DIN-5_180degree, J203 DIN-5_180degree, J204 DIN-5_180degree, J211 do not equip, J212 do not equip, J213 do not equip, J214 do not equip, J3 Conn_02x03_Odd_Even, J4 USB_B_Micro, J5 USB_B_Micro, J6 Conn_02x02_Odd_Even, J7 Conn_02x02_Odd_Even, J8 Conn_01x07, SW1 Rotary_Encoder_Switch, U1 74HCT245, U101 HCPL-2630, U102 HCPL-2630, U2 74HC595, U3 74HC165

Commit message: use proper IDC footprints for connectors
Parts:
- J2, J3: footprint Connector_PinHeader_2.54mm:PinHeader_2x03_P2.54mm_Vertical -> Connector_IDC:IDC-Header_2x03_P2.54mm_Vertical
Changed lines of the file:
@@
 F 0 "J2" H 10050 5575 50  0000 C CNN
 F 1 "Conn_02x03_Odd_Even" H 10050 5576 50  0001 C CNN
-F 2 "Connector_PinHeader_2.54mm:PinHeader_2x03_P2.54mm_Vertical" H 10000 5350 50  0001 C CNN
+F 2 "Connector_IDC:IDC-Header_2x03_P2.54mm_Vertical" H 10000 5350 50  0001 C CNN
 F 3 "~" H 10000 5350 50  0001 C CNN
 	1    10000 5350
@@
 F 0 "J3" H 10050 6300 50  0000 C CNN
 F 1 "Conn_02x03_Odd_Even" H 10050 6301 50  0001 C CNN
-F 2 "Connector_PinHeader_2.54mm:PinHeader_2x03_P2.54mm_Vertical" H 10000 6075 50  0001 C CNN
+F 2 "Connector_IDC:IDC-Header_2x03_P2.54mm_Vertical" H 10000 6075 50  0001 C CNN
 F 3 "~" H 10000 6075 50  0001 C CNN
 	1    10000 6075
@@
 todo: is BLK cheap to connect?
 $Comp
-L power:+3V3 #PWR?
+L power:+3V3 #PWR0116
 U 1 1 60E24BA6
 P 8675 4650
-F 0 "#PWR?" H 8675 4500 50  0001 C CNN
+F 0 "#PWR0116" H 8675 4500 50  0001 C CNN
 F 1 "+3V3" H 8550 4800 50  0000 C CNN
 F 2 "" H 8675 4650 50  0001 C CNN

Commit message: Fix silkscreen, final touches
Other:
- note removed: "todo (pcb): add jlcjlc marker to both"
- note removed: "todo (pcb): are the connectors oriented correctly?\ntodo (pcb): do the connector plugs fit?"
- note removed: "todo (pcb): mark pin 1 on connectors"
- note removed: "todo (pcb): move display up a little?"
- note removed: "todo: is BLK cheap to connect?"
Changed lines of the file:
@@
 NoConn ~ 825  7225
 NoConn ~ 9400 4600
-Text Notes 5975 -375 0    50   ~ 0
-todo: is BLK cheap to connect?
 $Comp
 L power:+3V3 #PWR0116
@@
 	1    0    0    -1
 $EndComp
-Text Notes 5975 -575 0    50   ~ 0
-todo (pcb): add jlcjlc marker to both
-Text Notes 5975 -475 0    50   ~ 0
-todo (pcb): move display up a little?
-Text Notes 5975 -850 0    50   ~ 0
-todo (pcb): mark pin 1 on connectors
-Text Notes 5975 -675 0    50   ~ 0
-todo (pcb): are the connectors oriented correctly?\ntodo (pcb): do the connector plugs fit?
 $Comp
 L Connector_Generic:Conn_02x03_Odd_Even J3

Commit message: Set the shift registers to a defined state as quick as possible after startup
Parts:
- R1: value R -> 10k
Changed lines of the file:
@@
 P 9375 825
 F 0 "R1" H 9445 871 50  0000 L CNN
-F 1 "R" H 9445 780 50  0000 L CNN
+F 1 "10k" H 9445 780 50  0000 L CNN
 F 2 "Resistor_SMD:R_0805_2012Metric" V 9305 825 50  0001 C CNN
 F 3 "~" H 9375 825 50  0001 C CNN
