File: schem/trs_pcb/trs_midi_output_8x.sch (KiCad schematic (older format))
At the start: 56 parts, among them J301 AudioJack3, J302 AudioJack3, J303 AudioJack3, J304 AudioJack3, J305 AudioJack3, J306 AudioJack3, J307 AudioJack3, J308 AudioJack3

Commit message: place components on trs pcb
Parts:
- J301, J302, J303, J304, J305, J306, J307, J308: footprint Connector_Audio:Jack_3.5mm_Ledino_KB3SPRS_Horizontal -> footprints:Jack_3.5mm_combo_ledino_upright
Changed lines of the file:
@@
 F 0 "J301" H 1800 1650 50  0000 R CNN
 F 1 "AudioJack3" H 2175 1350 50  0000 R CNN
-F 2 "Connector_Audio:Jack_3.5mm_Ledino_KB3SPRS_Horizontal" H 2050 1625 50  0001 C CNN
+F 2 "footprints:Jack_3.5mm_combo_ledino_upright" H 2050 1625 50  0001 C CNN
 F 3 "~" H 2050 1625 50  0001 C CNN
 	1    2050 1625
@@
 F 0 "J302" H 1800 2900 50  0000 R CNN
 F 1 "AudioJack3" H 2175 2600 50  0000 R CNN
-F 2 "Connector_Audio:Jack_3.5mm_Ledino_KB3SPRS_Horizontal" H 2050 2875 50  0001 C CNN
+F 2 "footprints:Jack_3.5mm_combo_ledino_upright" H 2050 2875 50  0001 C CNN
 F 3 "~" H 2050 2875 50  0001 C CNN
 	1    2050 2875
@@
 F 0 "J303" H 1800 4150 50  0000 R CNN
 F 1 "AudioJack3" H 2175 3850 50  0000 R CNN
-F 2 "Connector_Audio:Jack_3.5mm_Ledino_KB3SPRS_Horizontal" H 2050 4125 50  0001 C CNN
+F 2 "footprints:Jack_3.5mm_combo_ledino_upright" H 2050 4125 50  0001 C CNN
 F 3 "~" H 2050 4125 50  0001 C CNN
 	1    2050 4125
@@
 F 0 "J304" H 1800 5400 50  0000 R CNN
 F 1 "AudioJack3" H 2175 5100 50  0000 R CNN
-F 2 "Connector_Audio:Jack_3.5mm_Ledino_KB3SPRS_Horizontal" H 2050 5375 50  0001 C CNN
+F 2 "footprints:Jack_3.5mm_combo_ledino_upright" H 2050 5375 50  0001 C CNN
 F 3 "~" H 2050 5375 50  0001 C CNN
 	1    2050 5375
@@
 F 0 "J305" H 4175 1650 50  0000 R CNN
 F 1 "AudioJack3" H 4550 1350 50  0000 R CNN
-F 2 "Connector_Audio:Jack_3.5mm_Ledino_KB3SPRS_Horizontal" H 4425 1625 50  0001 C CNN
+F 2 "footprints:Jack_3.5mm_combo_ledino_upright" H 4425 1625 50  0001 C CNN
 F 3 "~" H 4425 1625 50  0001 C CNN
 	1    4425 1625
@@
 F 0 "J306" H 4175 2900 50  0000 R CNN
 F 1 "AudioJack3" H 4550 2600 50  0000 R CNN
-F 2 "Connector_Audio:Jack_3.5mm_Ledino_KB3SPRS_Horizontal" H 4425 2875 50  0001 C CNN
+F 2 "footprints:Jack_3.5mm_combo_ledino_upright" H 4425 2875 50  0001 C CNN
 F 3 "~" H 4425 2875 50  0001 C CNN
 	1    4425 2875
@@
 F 0 "J307" H 4175 4150 50  0000 R CNN
 F 1 "AudioJack3" H 4550 3850 50  0000 R CNN
-F 2 "Connector_Audio:Jack_3.5mm_Ledino_KB3SPRS_Horizontal" H 4425 4125 50  0001 C CNN
+F 2 "footprints:Jack_3.5mm_combo_ledino_upright" H 4425 4125 50  0001 C CNN
 F 3 "~" H 4425 4125 50  0001 C CNN
 	1    4425 4125
@@
 F 0 "J308" H 4175 5400 50  0000 R CNN
 F 1 "AudioJack3" H 4550 5100 50  0000 R CNN
-F 2 "Connector_Audio:Jack_3.5mm_Ledino_KB3SPRS_Horizontal" H 4425 5375 50  0001 C CNN
+F 2 "footprints:Jack_3.5mm_combo_ledino_upright" H 4425 5375 50  0001 C CNN
 F 3 "~" H 4425 5375 50  0001 C CNN
 	1    4425 5375
