File: schem/trs_pcb/trsmidi_input_8x.sch (KiCad schematic (older format))
At the start: 56 parts, among them J201 AudioJack3, J202 AudioJack3, J203 AudioJack3, J204 AudioJack3, J205 AudioJack3, J206 AudioJack3, J207 AudioJack3, J208 AudioJack3, U201 HCPL-2630, U202 HCPL-2630, U203 HCPL-2630, U204 HCPL-2630, U205 HCPL-2630, U206 HCPL-2630, U207 HCPL-2630, U208 HCPL-2630

Commit message: place components on trs pcb
Parts:
- J201, J202, J203, J204, J205, J206, J207, J208: footprint Connector_Audio:Jack_3.5mm_Ledino_KB3SPRS_Horizontal -> footprints:Jack_3.5mm_combo_ledino_upright
Changed lines of the file:
@@
 F 0 "J201" H 982 1725 50  0000 C CNN
 F 1 "AudioJack3" H 982 1634 50  0000 C CNN
-F 2 "Connector_Audio:Jack_3.5mm_Ledino_KB3SPRS_Horizontal" H 1000 1400 50  0001 C CNN
+F 2 "footprints:Jack_3.5mm_combo_ledino_upright" H 1000 1400 50  0001 C CNN
 F 3 "~" H 1000 1400 50  0001 C CNN
 	1    1000 1400
@@
 F 0 "J202" H 982 3300 50  0000 C CNN
 F 1 "AudioJack3" H 982 3209 50  0000 C CNN
-F 2 "Connector_Audio:Jack_3.5mm_Ledino_KB3SPRS_Horizontal" H 1000 2975 50  0001 C CNN
+F 2 "footprints:Jack_3.5mm_combo_ledino_upright" H 1000 2975 50  0001 C CNN
 F 3 "~" H 1000 2975 50  0001 C CNN
 	1    1000 2975
@@
 F 0 "J203" H 982 4875 50  0000 C CNN
 F 1 "AudioJack3" H 982 4784 50  0000 C CNN
-F 2 "Connector_Audio:Jack_3.5mm_Ledino_KB3SPRS_Horizontal" H 1000 4550 50  0001 C CNN
+F 2 "footprints:Jack_3.5mm_combo_ledino_upright" H 1000 4550 50  0001 C CNN
 F 3 "~" H 1000 4550 50  0001 C CNN
 	1    1000 4550
@@
 F 0 "J204" H 982 6450 50  0000 C CNN
 F 1 "AudioJack3" H 982 6359 50  0000 C CNN
-F 2 "Connector_Audio:Jack_3.5mm_Ledino_KB3SPRS_Horizontal" H 1000 6125 50  0001 C CNN
+F 2 "footprints:Jack_3.5mm_combo_ledino_upright" H 1000 6125 50  0001 C CNN
 F 3 "~" H 1000 6125 50  0001 C CNN
 	1    1000 6125
@@
 F 0 "J205" H 3732 1725 50  0000 C CNN
 F 1 "AudioJack3" H 3732 1634 50  0000 C CNN
-F 2 "Connector_Audio:Jack_3.5mm_Ledino_KB3SPRS_Horizontal" H 3750 1400 50  0001 C CNN
+F 2 "footprints:Jack_3.5mm_combo_ledino_upright" H 3750 1400 50  0001 C CNN
 F 3 "~" H 3750 1400 50  0001 C CNN
 	1    3750 1400
@@
 F 0 "J206" H 3732 3300 50  0000 C CNN
 F 1 "AudioJack3" H 3732 3209 50  0000 C CNN
-F 2 "Connector_Audio:Jack_3.5mm_Ledino_KB3SPRS_Horizontal" H 3750 2975 50  0001 C CNN
+F 2 "footprints:Jack_3.5mm_combo_ledino_upright" H 3750 2975 50  0001 C CNN
 F 3 "~" H 3750 2975 50  0001 C CNN
 	1    3750 2975
@@
 F 0 "J207" H 3732 4875 50  0000 C CNN
 F 1 "AudioJack3" H 3732 4784 50  0000 C CNN
-F 2 "Connector_Audio:Jack_3.5mm_Ledino_KB3SPRS_Horizontal" H 3750 4550 50  0001 C CNN
+F 2 "footprints:Jack_3.5mm_combo_ledino_upright" H 3750 4550 50  0001 C CNN
 F 3 "~" H 3750 4550 50  0001 C CNN
 	1    3750 4550
@@
 F 0 "J208" H 3732 6450 50  0000 C CNN
 F 1 "AudioJack3" H 3732 6359 50  0000 C CNN
-F 2 "Connector_Audio:Jack_3.5mm_Ledino_KB3SPRS_Horizontal" H 3750 6125 50  0001 C CNN
+F 2 "footprints:Jack_3.5mm_combo_ledino_upright" H 3750 6125 50  0001 C CNN
 F 3 "~" H 3750 6125 50  0001 C CNN
 	1    3750 6125
