File: schem/trs_pcb/pcb.kicad_pcb (KiCad board)
At the start: 2 copper layers, 124 parts, among them J101 2x3 female, J102 2x3 female, J201 AudioJack3, J202 AudioJack3, J203 AudioJack3, J204 AudioJack3, J205 AudioJack3, J206 AudioJack3, J207 AudioJack3, J208 AudioJack3, J301 AudioJack3, J302 AudioJack3, J303 AudioJack3, J304 AudioJack3, J305 AudioJack3, J306 AudioJack3, J307 AudioJack3, J308 AudioJack3, U101 74HCT245, U102 74HC165, U103 74HC595, U104 74HC595, U201 HCPL-2630, U202 HCPL-2630, U203 HCPL-2630, U204 HCPL-2630, U205 HCPL-2630, U206 HCPL-2630, U207 HCPL-2630, U208 HCPL-2630

Commit message: intermediate commit
Parts:
- added G***: LOGO, windfisch:windfisch_smaller, F.Cu at (128.8, 153.6)
- added J1: Conn_01x03_Male, Connector_PinHeader_2.54mm:PinHeader_1x03_P2.54mm_Horizontal, F.Cu at (138.3, 55.1)
- added J2: 2x3 female, Connector_PinHeader_2.54mm:PinHeader_2x03_P2.54mm_Vertical, F.Cu at (138.3, 155.1)
- added J3: 2x3 female, Connector_PinHeader_2.54mm:PinHeader_2x03_P2.54mm_Vertical, F.Cu at (143.3, 48.1)
- added REF**: MountingHole_3.2mm_M3_DIN965_Pad, MountingHole:MountingHole_3.2mm_M3_DIN965_Pad, F.Cu at (123.0, 41.3)
- added REF**: MountingHole_3.2mm_M3_DIN965, MountingHole:MountingHole_3.2mm_M3_DIN965, F.Cu at (118.3, 47.1)
- added REF**: MountingHole_3.2mm_M3_DIN965, MountingHole:MountingHole_3.2mm_M3_DIN965, F.Cu at (163.3, 154.1)
- added REF**: MountingHole_3.2mm_M3_DIN965, MountingHole:MountingHole_3.2mm_M3_DIN965, F.Cu at (118.3, 151.1)
- added REF**: MountingHole_3.2mm_M3_DIN965, MountingHole:MountingHole_3.2mm_M3_DIN965, F.Cu at (163.3, 49.1)
- added REF**: OSHW-Logo2_9.8x8mm_SilkScreen, Symbol:OSHW-Logo2_9.8x8mm_SilkScreen, F.Cu at (152.3, 154.6)
- moved D301 101.2 mm to (129.3, 68.4)
- moved D201 101.2 mm to (129.3, 57.8)
- moved D202 101.2 mm to (129.3, 84.8)
- moved D305 101.2 mm to (129.3, 73.8)
- moved R201 101.2 mm to (118.7, 51.6)
- moved R209 101.2 mm to (126.3, 57.2)
- moved J201 101.1 mm to (118.8, 61.1)
- moved J301 100.8 mm to (118.8, 73.3)
- moved J202 100.4 mm to (118.8, 85.6)
- moved J302 100.1 mm to (118.8, 97.8)
- moved J203 99.8 mm to (118.8, 110.1)
- moved J303 99.5 mm to (118.8, 122.3)
- moved J204 99.2 mm to (118.8, 134.6)
- moved J304 98.9 mm to (118.8, 146.8)
- moved REF** 78.9 mm to (100.7, 163.1)
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Routing:
- net (no net): track 0.00 -> 5.66 mm
- net Net-(J201-PadT): track 23.7 -> 20.8 mm
- net Net-(R214-Pad1): track 23.7 -> 20.9 mm
Other:
- board outline added: 56 x 115 mm
- board text added: "from master"

Commit message: Come layout considerations
Parts:
- moved J2 5.00 mm to (138.3, 150.1)
- moved G*** 4.50 mm to (128.8, 149.1)
- moved REF** 4.50 mm to (152.3, 150.1)
- moved REF** 3.00 mm to (163.3, 151.1)
- moved REF** 2.00 mm to (163.3, 47.1)
Other:
- board size 56 x 115 mm -> 56 x 110 mm
Changed lines of the file:
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@@
   (general
     (thickness 1.6)
-    (drawings 20)
+    (drawings 18)
     (tracks 235)
     (zones 0)
@@
   )
   (module MountingHole:MountingHole_3.2mm_M3_DIN965 (layer F.Cu)
-    (at 163.296 154.096)
+    (at 163.296 151.096)
     (descr "Mounting Hole 3.2mm, no annular, M3, DIN965")
     (tags "mounting hole 3.2mm no annular m3 din965")
@@
   )
   (module MountingHole:MountingHole_3.2mm_M3_DIN965 (layer F.Cu)
-    (at 163.296 49.096)
+    (at 163.296 47.096)
     (descr "Mounting Hole 3.2mm, no annular, M3, DIN965")
     (tags "mounting hole 3.2mm no annular m3 din965")
@@
   )
   (module Connector_PinHeader_2.54mm:PinHeader_2x03_P2.54mm_Vertical (layer F.Cu)
-    (at 138.256 155.096 90)
+    (at 138.256 150.096 90)
     (descr "Through hole straight pin header, 2x03, 2.54mm pitch, double rows")
     (tags "Through hole pin header THT 2x03 2.54mm double row")
@@
   )
   (module windfisch:windfisch_smaller (layer F.Cu)
-    (at 128.796 153.596)
+    (at 128.796 149.096)
     (fp_text reference G*** (at 0 0) (layer F.SilkS) hide
       (effects (font (size 1.524 1.524) (thickness 0.3)))
@@
   )
   (module Symbol:OSHW-Logo2_9.8x8mm_SilkScreen (layer F.Cu)
-    (at 152.296 154.596)
+    (at 152.296 150.096)
     (descr "Open Source Hardware Symbol")
     (tags "Logo Symbol OSHW")
@@
     )
   )
-  (gr_line (start 168.796 150.096) (end 168.796 155.096) (layer Edge.Cuts) (width 0.05))
-  (gr_line (start 112.796 150.096) (end 112.796 155.096) (layer Edge.Cuts) (width 0.05))
   (gr_line (start 145.296 45.596) (end 146.796 44.096) (layer Edge.Cuts) (width 0.05))
   (gr_line (start 134.796 44.096) (end 136.296 45.596) (layer Edge.Cuts) (width 0.05))
@@
     (effects (font (size 1 1) (thickness 0.15)))
   )
-  (gr_line (start 136.296 157.596) (end 145.296 157.596) (layer Edge.Cuts) (width 0.05))
+  (gr_line (start 136.296 152.596) (end 145.296 152.596) (layer Edge.Cuts) (width 0.05))
   (gr_line (start 112.796 48.096) (end 112.796 150.096) (layer Edge.Cuts) (width 0.05))
   (gr_arc (start 116.796 48.096) (end 116.796 44.096) (angle -90) (layer Edge.Cuts) (width 0.05))
-  (gr_line (start 134.796 159.096) (end 136.296 157.596) (layer Edge.Cuts) (width 0.05))
+  (gr_line (start 134.796 154.096) (end 136.296 152.596) (layer Edge.Cuts) (width 0.05))
   (gr_text "from master" (at 140.796 46.096) (layer B.SilkS)
     (effects (font (size 1 1) (thickness 0.15)) (justify mirror))
   )
   (gr_line (start 168.796 150.096) (end 168.796 48.096) (layer Edge.Cuts) (width 0.05))
-  (gr_arc (start 164.796 155.096) (end 164.796 159.096) (angle -90) (layer Edge.Cuts) (width 0.05))
+  (gr_arc (start 164.796 150.096) (end 164.796 154.096) (angle -90) (layer Edge.Cuts) (width 0.05))
   (gr_line (start 134.796 44.096) (end 116.796 44.096) (layer Edge.Cuts) (width 0.05))
   (gr_line (start 164.796 44.096) (end 146.796 44.096) (layer Edge.Cuts) (width 0.05))
-  (gr_line (start 145.296 157.596) (end 146.796 159.096) (layer Edge.Cuts) (width 0.05))
-  (gr_line (start 116.546 154.096) (end 134.546 154.096) (layer Edge.Cuts) (width 0.05))
+  (gr_line (start 145.296 152.596) (end 146.796 154.096) (layer Edge.Cuts) (width 0.05))
+  (gr_line (start 116.796 154.096) (end 134.796 154.096) (layer Edge.Cuts) (width 0.05))
   (gr_line (start 136.296 45.596) (end 145.296 45.596) (layer Edge.Cuts) (width 0.05))
   (gr_arc (start 164.796 48.096) (end 168.796 48.096) (angle -90) (layer Edge.Cuts) (width 0.05))
-  (gr_arc (start 116.796 155.096) (end 112.796 155.096) (angle -90) (layer Edge.Cuts) (width 0.05))
-  (gr_line (start 146.796 159.096) (end 164.796 159.096) (layer Edge.Cuts) (width 0.05))
+  (gr_arc (start 116.796 150.096) (end 112.796 150.096) (angle -90) (layer Edge.Cuts) (width 0.05))
+  (gr_line (start 146.796 154.096) (end 164.796 154.096) (layer Edge.Cuts) (width 0.05))
   (segment (start 42.7305 90.8095) (end 43.318 90.222) (width 0.25) (layer B.Cu) (net 1))
   (segment (start 41.198 90.8095) (end 42.7305 90.8095) (width 0.25) (layer B.Cu) (net 1))

Commit message: place components on trs pcb
Parts:
- removed A101: BluePill, footprints:BLUEPILL
- removed J1: Conn_01x03_Male, Connector_PinHeader_2.54mm:PinHeader_1x03_P2.54mm_Horizontal
- removed the J102 at (66.5, 113.0)
- removed J2: 2x3 female, Connector_PinHeader_2.54mm:PinHeader_2x03_P2.54mm_Vertical
- removed JP101: SolderJumper_3_Bridged12, Jumper:SolderJumper-3_P2.0mm_Open_TrianglePad1.0x1.5mm
- removed the REF** at (123.0, 41.3)
- removed the REF** at (100.7, 163.1)
- removed the REF** at (100.7, 48.8)
- removed U101: 74HCT245, Package_DIP:DIP-20_W7.62mm
- C202, C203, C204, C205, C206, C207, C208, D203, D204, D205, D206, D207, D208, D303, D304, D306, D307, D308, D309, D310, D311, D312, D313, D314, D315, D316, G***, R202, R203, R204, R206, R207, R208, R210, R211, R212, R213, R214, R215, R216, R217, R218, R219, R220, R221, R222, R223, R224, R301, R302, R303, R304, R305, R306, R307, R308, R309, R310, R311, R312, R313, R314, R315, R316, R317, R318, R319, R320, R321, R322, R323, R324, R325, R326, R327, R328, R329, R330, R331, R332: moved to B.Cu
- J101: value 2x3 female -> Conn_02x03_Odd_Even
- J102: renamed from J3; value 2x3 female -> Conn_02x03_Odd_Even
- J201, J202, J203, J204, J205, J206, J207, J208, J301, J302, J303, J304, J305, J306, J307, J308: footprint Connector_Audio:Jack_3.5mm_Ledino_KB3SPRS_Horizontal -> footprints:Jack_3.5mm_combo_ledino_upright
- moved D304 249.0 mm to (128.6, 140.9), turned to 90 degrees
- moved D308 243.4 mm to (128.6, 145.9), turned to 90 degrees
- moved D205 227.6 mm to (153.0, 140.5), turned to 270 degrees
- moved D303 223.7 mm to (128.6, 116.4), turned to 90 degrees
- moved D313 219.6 mm to (153.0, 125.7), turned to 270 degrees
- moved D206 215.4 mm to (153.0, 116.0), turned to 270 degrees
- moved R325 212.3 mm to (155.9, 130.6), turned to 180 degrees
- moved D307 210.9 mm to (128.6, 121.4), turned to 90 degrees
- moved D207 210.5 mm to (153.0, 91.5), turned to 270 degrees
- moved D306 208.9 mm to (128.6, 96.9), turned to 90 degrees
- moved R316 204.3 mm to (122.9, 146.8)
- moved D310 201.8 mm to (153.0, 106.2), turned to 270 degrees
- moved J305 199.4 mm to (162.8, 124.8), turned to 180 degrees
- moved R315 198.7 mm to (125.8, 141.0)
- moved R326 198.7 mm to (158.7, 124.9), turned to 180 degrees
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Connections:
- J101 pad 2: MIDI_MOSI_CHAIN -> MIDI_MISO_CHAIN
- J101 pad 3: SCK_MIDI_5 -> MIDI_MOSI_CHAIN
- J101 pad 4: GND -> STROBE_MIDI_5
- J101 pad 5: STROBE_MIDI_5 -> SCK_MIDI_5
- J101 pad 6: MIDI_MISO_CHAIN -> GND
- J102 pad 1: (no net) -> +5V
- J102 pad 2: (no net) -> MISO_MIDI
- J102 pad 3: (no net) -> MOSI_MIDI_5
- J102 pad 4: (no net) -> STROBE_MIDI_5
- J102 pad 5: (no net) -> SCK_MIDI_5
- J102 pad 6: (no net) -> GND
- J201 pad S: (no net) -> Net-(J201-PadS)
- J202 pad S: (no net) -> Net-(J202-PadS)
- J203 pad S: (no net) -> Net-(J203-PadS)
- J204 pad S: (no net) -> Net-(J204-PadS)
- J205 pad S: (no net) -> Net-(J205-PadS)
- J206 pad S: (no net) -> Net-(J206-PadS)
- J207 pad S: (no net) -> Net-(J207-PadS)
- J208 pad S: (no net) -> Net-(J208-PadS)
Routing:
- net GND: track 139.5 -> 0.00 mm, vias 1 -> 0
- net +5V: track 122.8 -> 0.00 mm, vias 3 -> 0
- net SCK_MIDI_5: track 63.8 -> 0.00 mm, vias 3 -> 0
- net MIDI_MOSI_CHAIN: track 63.8 -> 0.00 mm, vias 1 -> 0
- net MIDI_MISO_CHAIN: track 31.9 -> 0.00 mm, vias 1 -> 0
- net MISO_MIDI: track 30.3 -> 0.00 mm
- net Net-(A101-PadPA3): track 27.8 -> 0.00 mm, vias 2 -> 0
- net Net-(A101-PadPA5): track 27.4 -> 0.00 mm, vias 1 -> 0
- net STROBE_MIDI_5: track 26.7 -> 0.00 mm, vias 2 -> 0
- net Net-(J206-PadT): track 26.4 -> 0.00 mm
- net Net-(JP102-Pad2): track 23.9 -> 0.00 mm, vias 1 -> 0
- net /8x TRS Midi input/in5: track 23.8 -> 0.00 mm, vias 1 -> 0
- net Net-(A101-PadPA7): track 22.1 -> 0.00 mm, vias 2 -> 0
- net Net-(R214-Pad1): track 20.9 -> 0.00 mm
- net Net-(J201-PadT): track 20.8 -> 0.00 mm, vias 1 -> 0
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
Commit message: autorouted
Parts:
- JP102, R101: moved to B.Cu
- moved JP102 154.6 mm to (145.8, 121.7), turned to 180 degrees
- moved R101 124.6 mm to (148.8, 88.2), turned to 270 degrees
- renumbered REF** to hole1, REF** to hole2, REF** to hole3, REF** to hole4, REF** to oshw, G*** to wf
Routing:
- net +5V: track 0.00 -> 428.5 mm
- net GND: track 0.00 -> 422.8 mm, vias 0 -> 1
- net SCK_MIDI_5: track 0.00 -> 124.7 mm, vias 0 -> 1
- net STROBE_MIDI_5: track 0.00 -> 113.7 mm
- net /8x TRS Midi input/in3: track 0.00 -> 86.2 mm
- net /8x TRS Midi input/in5: track 0.00 -> 84.3 mm, vias 0 -> 1
- net /8x TRS Midi output/out7b: track 0.00 -> 81.5 mm
- net /8x TRS Midi input/in4: track 0.00 -> 76.5 mm, vias 0 -> 1
- net /8x TRS Midi input/in2: track 0.00 -> 72.6 mm
- net Net-(R216-Pad1): track 0.00 -> 71.3 mm
- net MIDI_MISO_CHAIN: track 0.00 -> 65.0 mm, vias 0 -> 1
- net MOSI_MIDI_5: track 0.00 -> 64.0 mm
- net Net-(R215-Pad1): track 0.00 -> 63.8 mm, vias 0 -> 2
- net /8x TRS Midi input/in7: track 0.00 -> 61.7 mm, vias 0 -> 1
- net /8x TRS Midi output/out7a: track 0.00 -> 60.3 mm
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- added copper zone on B.Cu, net GND
- added copper zone on F.Cu, net GND
Other:
- board text added: "Windfisch Enterprises"
- board text added: "https://github.com/ Windfisch/midikraken"
- board text added: "midikraken trs board (c) 2021 Florian Jung"
