File: schem/trs_pcb/pcb.kicad_pcb (KiCad board)
At the start: 2 copper layers, 56 x 110 mm, 125 parts, among them J101 Conn_02x03_Odd_Even, J102 Conn_02x03_Odd_Even, J201 AudioJack3, J202 AudioJack3, J203 AudioJack3, J204 AudioJack3, J205 AudioJack3, J206 AudioJack3, J207 AudioJack3, J208 AudioJack3, J301 AudioJack3, J302 AudioJack3, J303 AudioJack3, J304 AudioJack3, J305 AudioJack3, J306 AudioJack3, J307 AudioJack3, J308 AudioJack3, U102 74HC165, U103 74HC595, U104 74HC595, U201 HCPL-2630, U202 HCPL-2630, U203 HCPL-2630, U204 HCPL-2630, U205 HCPL-2630, U206 HCPL-2630, U207 HCPL-2630, U208 HCPL-2630

Commit message: move connectors inwards, reroute
Parts:
- J101, J102: footprint Connector_PinHeader_2.54mm:PinHeader_2x03_P2.54mm_Vertical -> Connector_IDC:IDC-Header_2x03_P2.54mm_Vertical
- moved C204 2.75 mm to (137.4, 139.8)
- moved C205 2.75 mm to (147.6, 139.9)
- moved R208 2.75 mm to (137.4, 134.8)
- moved R217 2.75 mm to (147.6, 134.9)
- moved U204 2.75 mm to (132.0, 133.6)
- moved U205 2.75 mm to (142.1, 133.6)
- moved C208 2.35 mm to (147.5, 63.5)
- moved R220 2.35 mm to (147.5, 58.2)
- moved U208 2.35 mm to (142.1, 56.9)
- moved C201 2.35 mm to (137.4, 63.4)
- moved R205 2.35 mm to (137.4, 58.2)
- moved U201 2.35 mm to (131.9, 56.9)
- moved C203 2.25 mm to (137.5, 128.7)
- moved C206 2.25 mm to (147.6, 128.6)
- moved R207 2.25 mm to (137.5, 123.4)
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Routing:
- net Net-(J203-PadT): track 41.1 -> 62.2 mm
- net /8x TRS Midi input/in5: track 84.3 -> 65.4 mm, vias 1 -> 0
- net Net-(J207-PadT): track 42.7 -> 61.6 mm, vias 0 -> 2
- net /8x TRS Midi input/in3: track 86.2 -> 101.7 mm
- net /8x TRS Midi input/in6: track 58.0 -> 48.0 mm
- net Net-(R203-Pad1): track 49.0 -> 57.5 mm, vias 0 -> 1
- net /8x TRS Midi output/out4b: track 32.2 -> 40.2 mm
- net /8x TRS Midi output/out1b: track 30.8 -> 23.2 mm
- net Net-(R204-Pad1): track 36.7 -> 29.8 mm, vias 0 -> 2
- net STROBE_MIDI_5: track 113.7 -> 120.6 mm
- net +5V: track 428.5 -> 423.8 mm
- net /8x TRS Midi output/out7a: track 60.3 -> 55.6 mm
- net Net-(R214-Pad1): track 50.7 -> 46.6 mm
- net /8x TRS Midi input/in7: track 61.7 -> 57.7 mm
- net Net-(R216-Pad1): track 71.3 -> 75.0 mm
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Other:
- board text added: "1"
- board text added: "2"
- board text added: "to slave"

Commit message: Fix silkscreen, final touches
Routing:
- net GND: track 424.5 -> 475.8 mm, vias 0 -> 3
Other:
- board text added: "JLCJLCJLCJLC"
- board text added: "midikraken trs board rev01 (c) 2021 Florian Jung"
- board text removed: "midikraken trs board (c) 2021 Florian Jung"
