File: schem/trs_pcb/pcb.sch (KiCad schematic (older format))
At the start: 10 parts, among them J101 2x3 female, J102 2x3 female, U101 74HCT245, U102 74HC165, U103 74HC595, U104 74HC595

Commit message: Come layout considerations
Parts:
- removed A101: BluePill, footprints:BLUEPILL, symbol bluepill:BluePill
- removed JP101: SolderJumper_3_Bridged12, Jumper:SolderJumper-3_P2.0mm_Open_TrianglePad1.0x1.5mm, symbol Jumper:SolderJumper_3_Bridged12
- removed U101: 74HCT245, Package_DIP:DIP-20_W7.62mm, symbol 74xx:74HC245
Connections:
- no-connect marks 6 -> 1
Other:
- note removed: "72HCT245 can be replaced by 74HCT541, but\npin 1 must be tied to GND instead of +5V then."
- moved on the sheet: R101, U102

Commit message: place components on trs pcb
Parts:
- removed J101, J102: 2x3 female, Connector_PinHeader_2.54mm:PinHeader_2x03_P2.54mm_Vertical, symbol Connector_Generic:Conn_02x03_Counter_Clockwise
- added J101, J102: Conn_02x03_Odd_Even, Connector_PinHeader_2.54mm:PinHeader_2x03_P2.54mm_Vertical, symbol Connector_Generic:Conn_02x03_Odd_Even
Connections:
- net +5V: now also J101.1 (Pin_1), J102.1 (Pin_1)
- net GND: now also J101.6 (Pin_6), J102.6 (Pin_6)
- net MIDI_MISO_CHAIN: now also J101.2 (Pin_2)
- net MIDI_MOSI_CHAIN: now also J101.3 (Pin_3)
- net MISO_MIDI: now also J102.2 (Pin_2)
- net MOSI_MIDI_5: now also J102.3 (Pin_3)
- net SCK_MIDI_5: now also J101.5 (Pin_5), J102.5 (Pin_5)
- net STROBE_MIDI_5: now also J101.4 (Pin_4), J102.4 (Pin_4)
Changed lines of the file:
@@
 NoConn ~ 4675 1725
-$Comp
-L Connector_Generic:Conn_02x03_Counter_Clockwise J101
-U 1 1 60B33612
-P 9700 5325
-F 0 "J101" H 9750 5600 50  0000 C CNN
-F 1 "2x3 female" H 9675 5100 50  0000 C CNN
-F 2 "Connector_PinHeader_2.54mm:PinHeader_2x03_P2.54mm_Vertical" H 9700 5325 50  0001 C CNN
-F 3 "~" H 9700 5325 50  0001 C CNN
-	1    9700 5325
-	1    0    0    -1
-$EndComp
 $Comp
 L power:+5V #PWR0115
@@
 P 10000 5425
 F 0 "#PWR0117" H 10000 5175 50  0001 C CNN
-F 1 "GND" H 10005 5252 50  0000 C CNN
+F 1 "GND" H 10150 5350 50  0000 C CNN
 F 2 "" H 10000 5425 50  0001 C CNN
 F 3 "" H 10000 5425 50  0001 C CNN
@@
 Text GLabel 9500 5425 0    50   Input ~ 0
 SCK_MIDI_5
-Text Notes 9325 5650 0    50   ~ 0
+Text Notes 9475 5625 0    50   ~ 0
 chain to slave
-$Comp
-L Connector_Generic:Conn_02x03_Counter_Clockwise J102
-U 1 1 60B5097F
-P 9700 6050
-F 0 "J102" H 9750 6325 50  0000 C CNN
-F 1 "2x3 female" H 9675 5825 50  0000 C CNN
-F 2 "Connector_PinHeader_2.54mm:PinHeader_2x03_P2.54mm_Vertical" H 9700 6050 50  0001 C CNN
-F 3 "~" H 9700 6050 50  0001 C CNN
-	1    9700 6050
-	1    0    0    -1
-$EndComp
 $Comp
 L power:+5V #PWR0116
@@
 P 10000 6150
 F 0 "#PWR0118" H 10000 5900 50  0001 C CNN
-F 1 "GND" H 10005 5977 50  0000 C CNN
+F 1 "GND" H 10150 6075 50  0000 C CNN
 F 2 "" H 10000 6150 50  0001 C CNN
 F 3 "" H 10000 6150 50  0001 C CNN
@@
 Text GLabel 9500 6150 0    50   Input ~ 0
 SCK_MIDI_5
-Text Notes 9325 6375 0    50   ~ 0
+Text Notes 9400 6375 0    50   ~ 0
 chain from master
 Text GLabel 9500 6050 0    50   Input ~ 0
@@
 	1    0    0    -1
 $EndComp
+$Comp
+L Connector_Generic:Conn_02x03_Odd_Even J101
+U 1 1 60C0AEA7
+P 9700 5325
+F 0 "J101" H 9750 5550 50  0000 C CNN
+F 1 "Conn_02x03_Odd_Even" H 9750 5551 50  0001 C CNN
+F 2 "Connector_PinHeader_2.54mm:PinHeader_2x03_P2.54mm_Vertical" H 9700 5325 50  0001 C CNN
+F 3 "~" H 9700 5325 50  0001 C CNN
+	1    9700 5325
+	1    0    0    -1
+$EndComp
+$Comp
+L Connector_Generic:Conn_02x03_Odd_Even J102
+U 1 1 60C0CBEA
+P 9700 6050
+F 0 "J102" H 9750 6275 50  0000 C CNN
+F 1 "Conn_02x03_Odd_Even" H 9750 6276 50  0001 C CNN
+F 2 "Connector_PinHeader_2.54mm:PinHeader_2x03_P2.54mm_Vertical" H 9700 6050 50  0001 C CNN
+F 3 "~" H 9700 6050 50  0001 C CNN
+	1    9700 6050
+	1    0    0    -1
+$EndComp

Commit message: use proper IDC footprints for connectors
Parts:
- J101, J102: footprint Connector_PinHeader_2.54mm:PinHeader_2x03_P2.54mm_Vertical -> Connector_IDC:IDC-Header_2x03_P2.54mm_Vertical
Changed lines of the file:
@@
 F 0 "J101" H 9750 5550 50  0000 C CNN
 F 1 "Conn_02x03_Odd_Even" H 9750 5551 50  0001 C CNN
-F 2 "Connector_PinHeader_2.54mm:PinHeader_2x03_P2.54mm_Vertical" H 9700 5325 50  0001 C CNN
+F 2 "Connector_IDC:IDC-Header_2x03_P2.54mm_Vertical" H 9700 5325 50  0001 C CNN
 F 3 "~" H 9700 5325 50  0001 C CNN
 	1    9700 5325
@@
 F 0 "J102" H 9750 6275 50  0000 C CNN
 F 1 "Conn_02x03_Odd_Even" H 9750 6276 50  0001 C CNN
-F 2 "Connector_PinHeader_2.54mm:PinHeader_2x03_P2.54mm_Vertical" H 9700 6050 50  0001 C CNN
+F 2 "Connector_IDC:IDC-Header_2x03_P2.54mm_Vertical" H 9700 6050 50  0001 C CNN
 F 3 "~" H 9700 6050 50  0001 C CNN
 	1    9700 6050
