File: hardware/din5_pcb/din5_pcb.kicad_pcb (KiCad board)
At the start: 2 copper layers, 56 x 110 mm, 82 parts, among them J1 Conn_01x03_Male, J101 DIN-5_180degree, J102 DIN-5_180degree, J103 DIN-5_180degree, J104 DIN-5_180degree, J111 do not equip, J112 do not equip, J113 do not equip, J114 do not equip, J2 Conn_02x03_Odd_Even, J201 DIN-5_180degree, J202 DIN-5_180degree, J203 DIN-5_180degree, J204 DIN-5_180degree, J211 do not equip, J212 do not equip, J213 do not equip, J214 do not equip, J3 Conn_02x03_Odd_Even, J4 USB_B_Micro, J5 USB_B_Micro, J6 Conn_02x02_Odd_Even, J7 Conn_02x02_Odd_Even, J8 Conn_01x07, SW1 Rotary_Encoder_Switch, U1 74HCT245, U101 HCPL-2630, U102 HCPL-2630, U2 74HC595, U3 74HC165

Commit message: Convert din5_pcb.kicad_pcb to KiCAD 6 format
Other:
- net class Default removed
