File: hardware/din5_pcb/din5_pcb.sch (KiCad schematic (older format))
At the start: 76 parts, among them J1 Conn_01x03_Male, J101 DIN-5_180degree, J102 DIN-5_180degree, J103 DIN-5_180degree, J104 DIN-5_180degree, J111 do not equip, J112 do not equip, J113 do not equip, J114 do not equip, J2 Conn_02x03_Odd_Even, J201 DIN-5_180degree, J202 DIN-5_180degree, J203 DIN-5_180degree, J204 DIN-5_180degree, J211 do not equip, J212 do not equip, J213 do not equip, J214 do not equip, J3 Conn_02x03_Odd_Even, J4 USB_B_Micro, J5 USB_B_Micro, J6 Conn_02x02_Odd_Even, J7 Conn_02x02_Odd_Even, J8 Conn_01x07, SW1 Rotary_Encoder_Switch, U1 74HCT245, U101 HCPL-2630, U102 HCPL-2630, U2 74HC595, U3 74HC165

Commit message: Add license hints to all hardware files
Parts:
- A1: symbol bluepill:BluePill -> din5_pcb-rescue:BluePill-bluepill
Other:
- note added: "Copyright (c) 2021 Florian Jung.\n\nThis source describes Open Hardware and is licensed under the CERN-OHL-S v2.\n\nYou may redistribute and modify this source and make products using it under\nthe terms of the CERN-OHL-S v2 (https://ohwr.org/cern_ohl_s_v2.txt).\n\nThis source is distributed WITHOUT ANY EXPRESS OR IMPLIED WARRANTY,\nINCLUDING OF MERCHANTABILITY, SATISFACTORY QUALITY AND FITNESS F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"
- moved on the sheet: J2, J3, J4, J5, J6, J7, J8, JP14, R1, SW1, U2, U3

Commit message: Bill of material
Parts:
- D101, D102, D103, D104: value LED -> green
- D201, D202, D203, D204: value yellow -> red
- J1: value Conn_01x03_Male -> pin header 1x3 angled
- J101, J102, J103, J104, J201, J202, J203, J204: value DIN-5_180degree -> DS-5-01
- J2, J3: value Conn_02x03_Odd_Even -> WSL 6G (box connector 6 pin)
- J4, J5: value USB_B_Micro -> (USB_B_Micro)
- J6, J7: value Conn_02x02_Odd_Even -> (pin header 2x2)
- J8: value Conn_01x07 -> pin socket 1x7
- SW1: value Rotary_Encoder_Switch -> EC11 rotary encoder with push button
Changed lines of the file:
@@
 AR Path="/60D537D8" Ref="J204"  Part="1"
 F 0 "J204" H 5625 7150 50  0000 C CNN
-F 1 "DIN-5_180degree" H 5675 6975 50  0000 C CNN
+F 1 "DS-5-01" H 5675 6975 50  0000 C CNN
 F 2 "footprints:DIN5" H 5675 7225 50  0001 C CNN
 F 3 "http://www.mouser.com/ds/2/18/40_c091_abd_e-75918.pdf" H 5675 7225 50  0001 C CNN
@@
 AR Path="/60D537FB" Ref="D204"  Part="1"
 F 0 "D204" V 4525 6975 50  0000 L CNN
-F 1 "yellow" V 4450 6950 50  0000 L CNN
+F 1 "red" V 4450 6950 50  0000 L CNN
 F 2 "LED_THT:LED_D3.0mm_Horizontal_O3.81mm_Z6.0mm" H 4500 7275 50  0001 C CNN
 F 3 "~" H 4500 7275 50  0001 C CNN
@@
 AR Path="/60D53814" Ref="J203"  Part="1"
 F 0 "J203" H 5625 6150 50  0000 C CNN
-F 1 "DIN-5_180degree" H 5675 5975 50  0000 C CNN
+F 1 "DS-5-01" H 5675 5975 50  0000 C CNN
 F 2 "footprints:DIN5" H 5675 6225 50  0001 C CNN
 F 3 "http://www.mouser.com/ds/2/18/40_c091_abd_e-75918.pdf" H 5675 6225 50  0001 C CNN
@@
 AR Path="/60D53837" Ref="D203"  Part="1"
 F 0 "D203" V 4525 5975 50  0000 L CNN
-F 1 "yellow" V 4450 5950 50  0000 L CNN
+F 1 "red" V 4450 5950 50  0000 L CNN
 F 2 "LED_THT:LED_D3.0mm_Horizontal_O3.81mm_Z6.0mm" H 4500 6275 50  0001 C CNN
 F 3 "~" H 4500 6275 50  0001 C CNN
@@
 AR Path="/60D53850" Ref="J202"  Part="1"
 F 0 "J202" H 5625 5150 50  0000 C CNN
-F 1 "DIN-5_180degree" H 5675 4975 50  0000 C CNN
+F 1 "DS-5-01" H 5675 4975 50  0000 C CNN
 F 2 "footprints:DIN5" H 5675 5225 50  0001 C CNN
 F 3 "http://www.mouser.com/ds/2/18/40_c091_abd_e-75918.pdf" H 5675 5225 50  0001 C CNN
@@
 AR Path="/60D53873" Ref="D202"  Part="1"
 F 0 "D202" V 4525 4975 50  0000 L CNN
-F 1 "yellow" V 4450 4950 50  0000 L CNN
+F 1 "red" V 4450 4950 50  0000 L CNN
 F 2 "LED_THT:LED_D3.0mm_Horizontal_O3.81mm_Z6.0mm" H 4500 5275 50  0001 C CNN
 F 3 "~" H 4500 5275 50  0001 C CNN
@@
 AR Path="/60D5388C" Ref="J201"  Part="1"
 F 0 "J201" H 5625 4150 50  0000 C CNN
-F 1 "DIN-5_180degree" H 5675 3975 50  0000 C CNN
+F 1 "DS-5-01" H 5675 3975 50  0000 C CNN
 F 2 "footprints:DIN5" H 5675 4225 50  0001 C CNN
 F 3 "http://www.mouser.com/ds/2/18/40_c091_abd_e-75918.pdf" H 5675 4225 50  0001 C CNN
@@
 AR Path="/60D538AF" Ref="D201"  Part="1"
 F 0 "D201" V 4525 3975 50  0000 L CNN
-F 1 "yellow" V 4450 3950 50  0000 L CNN
+F 1 "red" V 4450 3950 50  0000 L CNN
 F 2 "LED_THT:LED_D3.0mm_Horizontal_O3.81mm_Z6.0mm" H 4500 4275 50  0001 C CNN
 F 3 "~" H 4500 4275 50  0001 C CNN
@@
 P 3100 1850
 F 0 "J1" V 3162 1662 50  0000 R CNN
-F 1 "Conn_01x03_Male" V 3253 1662 50  0001 R CNN
+F 1 "pin header 1x3 angled" V 3253 1662 50  0001 R CNN
 F 2 "Connector_PinHeader_2.54mm:PinHeader_1x03_P2.54mm_Horizontal" H 3100 1850 50  0001 C CNN
 F 3 "~" H 3100 1850 50  0001 C CNN
@@
 AR Path="/60B6A74D/60D3D107" Ref="D?"  Part="1"
 F 0 "D101" V 3550 4175 50  0000 R CNN
-F 1 "LED" V 3475 4150 50  0000 R CNN
+F 1 "green" V 3475 4150 50  0000 R CNN
 F 2 "LED_THT:LED_D3.0mm_Horizontal_O1.27mm_Z2.0mm" H 3275 4075 50  0001 C CNN
 F 3 "~" H 3275 4075 50  0001 C CNN
@@
 AR Path="/60B6A74D/60D3D13A" Ref="D?"  Part="1"
 F 0 "D102" V 4225 4175 50  0000 R CNN
-F 1 "LED" V 4150 4150 50  0000 R CNN
+F 1 "green" V 4150 4150 50  0000 R CNN
 F 2 "LED_THT:LED_D3.0mm_Horizontal_O1.27mm_Z2.0mm" H 3950 4075 50  0001 C CNN
 F 3 "~" H 3950 4075 50  0001 C CNN
@@
 AR Path="/60B6A74D/60D3D1C0" Ref="D?"  Part="1"
 F 0 "D104" V 4250 6100 50  0000 R CNN
-F 1 "LED" V 4175 6075 50  0000 R CNN
+F 1 "green" V 4175 6075 50  0000 R CNN
 F 2 "LED_THT:LED_D3.0mm_Horizontal_O1.27mm_Z2.0mm" H 3950 6000 50  0001 C CNN
 F 3 "~" H 3950 6000 50  0001 C CNN
@@
 AR Path="/60B6A74D/60D3D18D" Ref="D?"  Part="1"
 F 0 "D103" V 3575 6100 50  0000 R CNN
-F 1 "LED" V 3500 6075 50  0000 R CNN
+F 1 "green" V 3500 6075 50  0000 R CNN
 F 2 "LED_THT:LED_D3.0mm_Horizontal_O1.27mm_Z2.0mm" H 3275 6000 50  0001 C CNN
 F 3 "~" H 3275 6000 50  0001 C CNN
@@
 P 8025 2950
 F 0 "J5" H 8082 3417 50  0000 C CNN
-F 1 "USB_B_Micro" H 8082 3326 50  0000 C CNN
+F 1 "(USB_B_Micro)" H 8082 3326 50  0000 C CNN
 F 2 "Connector_USB:USB_Micro-B_Wuerth_629105150521" H 8175 2900 50  0001 C CNN
 F 3 "~" H 8175 2900 50  0001 C CNN
@@
 AR Path="/60D3D1E5" Ref="J104"  Part="1"
 F 0 "J104" H 1400 7150 50  0000 C CNN
-F 1 "DIN-5_180degree" H 1550 7400 50  0000 C CNN
+F 1 "DS-5-01" H 1550 7400 50  0000 C CNN
 F 2 "footprints:DIN5" H 1550 6925 50  0001 C CNN
 F 3 "http://www.mouser.com/ds/2/18/40_c091_abd_e-75918.pdf" H 1550 6925 50  0001 C CNN
@@
 AR Path="/60D3D1D9" Ref="J103"  Part="1"
 F 0 "J103" H 1400 6300 50  0000 C CNN
-F 1 "DIN-5_180degree" H 1550 5825 50  0000 C CNN
+F 1 "DS-5-01" H 1550 5825 50  0000 C CNN
 F 2 "footprints:DIN5" H 1550 6075 50  0001 C CNN
 F 3 "http://www.mouser.com/ds/2/18/40_c091_abd_e-75918.pdf" H 1550 6075 50  0001 C CNN
@@
 AR Path="/60D3D15F" Ref="J102"  Part="1"
 F 0 "J102" H 1400 5225 50  0000 C CNN
-F 1 "DIN-5_180degree" H 1550 5475 50  0000 C CNN
+F 1 "DS-5-01" H 1550 5475 50  0000 C CNN
 F 2 "footprints:DIN5" H 1550 5000 50  0001 C CNN
 F 3 "http://www.mouser.com/ds/2/18/40_c091_abd_e-75918.pdf" H 1550 5000 50  0001 C CNN
@@
 AR Path="/60D3D153" Ref="J101"  Part="1"
 F 0 "J101" H 1400 4375 50  0000 C CNN
-F 1 "DIN-5_180degree" H 1550 3900 50  0000 C CNN
+F 1 "DS-5-01" H 1550 3900 50  0000 C CNN
 F 2 "footprints:DIN5" H 1550 4150 50  0001 C CNN
 F 3 "http://www.mouser.com/ds/2/18/40_c091_abd_e-75918.pdf" H 1550 4150 50  0001 C CNN
@@
 P 5875 2950
 F 0 "J4" H 5932 3417 50  0000 C CNN
-F 1 "USB_B_Micro" H 5932 3326 50  0000 C CNN
+F 1 "(USB_B_Micro)" H 5932 3326 50  0000 C CNN
 F 2 "Connector_USB:USB_Micro-B_Wuerth_629105150521" H 6025 2900 50  0001 C CNN
 F 3 "~" H 6025 2900 50  0001 C CNN
@@
 P 8650 3050
 F 0 "J7" H 8700 3175 50  0000 C CNN
-F 1 "Conn_02x02_Odd_Even" H 8700 3176 50  0001 C CNN
+F 1 "(pin header 2x2)" H 8700 3176 50  0001 C CNN
 F 2 "Connector_PinHeader_2.54mm:PinHeader_2x02_P2.54mm_Vertical" H 8650 3050 50  0001 C CNN
 F 3 "~" H 8650 3050 50  0001 C CNN
@@
 P 6825 2900
 F 0 "J6" H 6875 3025 50  0000 C CNN
-F 1 "Conn_02x02_Odd_Even" H 6875 3026 50  0001 C CNN
+F 1 "(pin header 2x2)" H 6875 3026 50  0001 C CNN
 F 2 "Connector_PinHeader_2.54mm:PinHeader_2x02_P2.54mm_Vertical" H 6825 2900 50  0001 C CNN
 F 3 "~" H 6825 2900 50  0001 C CNN
@@
 P 10625 2950
 F 0 "SW1" H 10625 3317 50  0000 C CNN
-F 1 "Rotary_Encoder_Switch" H 10625 3226 50  0000 C CNN
+F 1 "EC11 rotary encoder with push button" H 10750 3225 50  0000 C CNN
 F 2 "Rotary_Encoder:RotaryEncoder_Alps_EC11E-Switch_Vertical_H20mm" H 10475 3110 50  0001 C CNN
 F 3 "~" H 10625 3210 50  0001 C CNN
@@
 P 7775 4400
 F 0 "J8" V 7693 4012 50  0000 R CNN
-F 1 "Conn_01x07" V 7648 4012 50  0001 R CNN
+F 1 "pin socket 1x7" V 7648 4012 50  0001 R CNN
 F 2 "Connector_PinHeader_2.54mm:PinHeader_1x07_P2.54mm_Vertical" H 7775 4400 50  0001 C CNN
 F 3 "~" H 7775 4400 50  0001 C CNN
@@
 P 10175 4550
 F 0 "J3" H 10225 4775 50  0000 C CNN
-F 1 "Conn_02x03_Odd_Even" H 10225 4776 50  0001 C CNN
+F 1 "WSL 6G (box connector 6 pin)" H 10225 4776 50  0001 C CNN
 F 2 "Connector_IDC:IDC-Header_2x03_P2.54mm_Vertical" H 10175 4550 50  0001 C CNN
 F 3 "~" H 10175 4550 50  0001 C CNN
@@
 P 10175 3825
 F 0 "J2" H 10225 4050 50  0000 C CNN
-F 1 "Conn_02x03_Odd_Even" H 10225 4051 50  0001 C CNN
+F 1 "WSL 6G (box connector 6 pin)" H 10225 4051 50  0001 C CNN
 F 2 "Connector_IDC:IDC-Header_2x03_P2.54mm_Vertical" H 10175 3825 50  0001 C CNN
 F 3 "~" H 10175 3825 50  0001 C CNN

Commit message: Change LED resistors from 1k to 220 Ohm.
Closes #61.
Parts:
- R201, R202, R203, R204: value 1k -> 220
Changed lines of the file:
@@
 AR Path="/60D537F5" Ref="R204"  Part="1"
 F 0 "R204" H 4575 6975 50  0000 L CNN
-F 1 "1k" V 4500 6925 50  0000 L CNN
+F 1 "220" V 4500 6900 50  0000 L CNN
 F 2 "Resistor_SMD:R_0805_2012Metric" V 4430 6975 50  0001 C CNN
 F 3 "~" H 4500 6975 50  0001 C CNN
@@
 AR Path="/60D53831" Ref="R203"  Part="1"
 F 0 "R203" H 4575 5975 50  0000 L CNN
-F 1 "1k" V 4500 5925 50  0000 L CNN
+F 1 "220" V 4500 5900 50  0000 L CNN
 F 2 "Resistor_SMD:R_0805_2012Metric" V 4430 5975 50  0001 C CNN
 F 3 "~" H 4500 5975 50  0001 C CNN
@@
 AR Path="/60D5386D" Ref="R202"  Part="1"
 F 0 "R202" H 4575 4975 50  0000 L CNN
-F 1 "1k" V 4500 4925 50  0000 L CNN
+F 1 "220" V 4500 4900 50  0000 L CNN
 F 2 "Resistor_SMD:R_0805_2012Metric" V 4430 4975 50  0001 C CNN
 F 3 "~" H 4500 4975 50  0001 C CNN
@@
 AR Path="/60D538A9" Ref="R201"  Part="1"
 F 0 "R201" H 4575 3975 50  0000 L CNN
-F 1 "1k" V 4500 3925 50  0000 L CNN
+F 1 "220" V 4500 3900 50  0000 L CNN
 F 2 "Resistor_SMD:R_0805_2012Metric" V 4430 3975 50  0001 C CNN
 F 3 "~" H 4500 3975 50  0001 C CNN

Commit message: Fix LED colors, add interactive bom
Parts:
- D101, D102, D103, D104: value green -> red
- D201, D202, D203, D204: value red -> green
Changed lines of the file:
@@
 AR Path="/60D537FB" Ref="D204"  Part="1"
 F 0 "D204" V 4525 6975 50  0000 L CNN
-F 1 "red" V 4450 6950 50  0000 L CNN
+F 1 "green" V 4450 6950 50  0000 L CNN
 F 2 "LED_THT:LED_D3.0mm_Horizontal_O3.81mm_Z6.0mm" H 4500 7275 50  0001 C CNN
 F 3 "~" H 4500 7275 50  0001 C CNN
@@
 AR Path="/60D53837" Ref="D203"  Part="1"
 F 0 "D203" V 4525 5975 50  0000 L CNN
-F 1 "red" V 4450 5950 50  0000 L CNN
+F 1 "green" V 4450 5950 50  0000 L CNN
 F 2 "LED_THT:LED_D3.0mm_Horizontal_O3.81mm_Z6.0mm" H 4500 6275 50  0001 C CNN
 F 3 "~" H 4500 6275 50  0001 C CNN
@@
 AR Path="/60D53873" Ref="D202"  Part="1"
 F 0 "D202" V 4525 4975 50  0000 L CNN
-F 1 "red" V 4450 4950 50  0000 L CNN
+F 1 "green" V 4450 4950 50  0000 L CNN
 F 2 "LED_THT:LED_D3.0mm_Horizontal_O3.81mm_Z6.0mm" H 4500 5275 50  0001 C CNN
 F 3 "~" H 4500 5275 50  0001 C CNN
@@
 AR Path="/60D538AF" Ref="D201"  Part="1"
 F 0 "D201" V 4525 3975 50  0000 L CNN
-F 1 "red" V 4450 3950 50  0000 L CNN
+F 1 "green" V 4450 3950 50  0000 L CNN
 F 2 "LED_THT:LED_D3.0mm_Horizontal_O3.81mm_Z6.0mm" H 4500 4275 50  0001 C CNN
 F 3 "~" H 4500 4275 50  0001 C CNN
@@
 AR Path="/60B6A74D/60D3D107" Ref="D?"  Part="1"
 F 0 "D101" V 3550 4175 50  0000 R CNN
-F 1 "green" V 3475 4150 50  0000 R CNN
+F 1 "red" V 3475 4150 50  0000 R CNN
 F 2 "LED_THT:LED_D3.0mm_Horizontal_O1.27mm_Z2.0mm" H 3275 4075 50  0001 C CNN
 F 3 "~" H 3275 4075 50  0001 C CNN
@@
 AR Path="/60B6A74D/60D3D13A" Ref="D?"  Part="1"
 F 0 "D102" V 4225 4175 50  0000 R CNN
-F 1 "green" V 4150 4150 50  0000 R CNN
+F 1 "red" V 4150 4150 50  0000 R CNN
 F 2 "LED_THT:LED_D3.0mm_Horizontal_O1.27mm_Z2.0mm" H 3950 4075 50  0001 C CNN
 F 3 "~" H 3950 4075 50  0001 C CNN
@@
 AR Path="/60B6A74D/60D3D1C0" Ref="D?"  Part="1"
 F 0 "D104" V 4250 6100 50  0000 R CNN
-F 1 "green" V 4175 6075 50  0000 R CNN
+F 1 "red" V 4175 6075 50  0000 R CNN
 F 2 "LED_THT:LED_D3.0mm_Horizontal_O1.27mm_Z2.0mm" H 3950 6000 50  0001 C CNN
 F 3 "~" H 3950 6000 50  0001 C CNN
@@
 AR Path="/60B6A74D/60D3D18D" Ref="D?"  Part="1"
 F 0 "D103" V 3575 6100 50  0000 R CNN
-F 1 "green" V 3500 6075 50  0000 R CNN
+F 1 "red" V 3500 6075 50  0000 R CNN
 F 2 "LED_THT:LED_D3.0mm_Horizontal_O1.27mm_Z2.0mm" H 3275 6000 50  0001 C CNN
 F 3 "~" H 3275 6000 50  0001 C CNN
