File: hardware/trs_pcb/pcb.kicad_pcb (KiCad board)
At the start: 2 copper layers, 56 x 110 mm, 125 parts, among them J101 Conn_02x03_Odd_Even, J102 Conn_02x03_Odd_Even, J201 AudioJack3, J202 AudioJack3, J203 AudioJack3, J204 AudioJack3, J205 AudioJack3, J206 AudioJack3, J207 AudioJack3, J208 AudioJack3, J301 AudioJack3, J302 AudioJack3, J303 AudioJack3, J304 AudioJack3, J305 AudioJack3, J306 AudioJack3, J307 AudioJack3, J308 AudioJack3, U102 74HC165, U103 74HC595, U104 74HC595, U201 HCPL-2630, U202 HCPL-2630, U203 HCPL-2630, U204 HCPL-2630, U205 HCPL-2630, U206 HCPL-2630, U207 HCPL-2630, U208 HCPL-2630

Commit message: Add license hints to all hardware files
Other:
- board text added: "Copyright (c) 2021 Florian Jung. This source describes Open Hardware and is licensed under the CERN-OHL-S v2. You may redistribute and modify this source and make products using it under the terms of the CERN-OHL-S v2 (https://ohwr.org/cern_ohl_s_v2.txt). This source is distributed WITHOUT ANY EXPRESS OR IMPLIED WARRANTY, INCLUDING OF MERCHANTABILITY, SATISFACTORY QUALITY AND FITNESS FOR A PARTIC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"
Changed lines of the file:
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@@
   (general
     (thickness 1.6)
-    (drawings 31)
+    (drawings 32)
     (tracks 1506)
     (zones 0)
@@
   )
   (page A4)
+  (title_block
+    (title "Midikraken TRS")
+    (rev 01)
+    (company Windfisch)
+    (comment 1 "Copyright (c) 2021 Florian Jung.\n")
+    (comment 2 "the terms of the CERN-OHL-S v2 (https://ohwr.org/cern_ohl_s_v2.txt).\n")
+    (comment 3 "You may redistribute and modify this source and make products using it under\n")
+    (comment 4 "This source describes Open Hardware and is licensed under the CERN-OHL-S v2.\n")
+  )
   (layers
     (0 F.Cu signal)
@@
     )
   )
+  (gr_text "Copyright (c) 2021 Florian Jung.\n\nThis source describes Open Hardware and is licensed under the CERN-OHL-S v2.\n\nYou may redistribute and modify this source and make products using it under\nthe terms of the CERN-OHL-S v2 (https://ohwr.org/cern_ohl_s_v2.txt).\n\nThis source is distributed WITHOUT ANY EXPRESS OR IMPLIED WARRANTY,\nINCLUDING OF MERCHANTABILITY, SATISFACTORY QUALITY AND FITNESS FOR A\nPARTICULAR PURPOSE. Please see the CERN-OHL-S v2 for applicable conditions.\n\nSource location: https://github.com/Windfisch/midikraken\n\nAs per CERN-OHL-S v2 section 4, should You produce hardware based on this\nsource, You must where practicable maintain the Source Location visible\non the external case of the Gizmo or other products you make using this\nsource.\n" (at 186.766 140.386) (layer Cmts.User)
+    (effects (font (size 1.5 1.5) (thickness 0.15)) (justify left))
+  )
   (gr_text JLCJLCJLCJLC (at 125.966 151.386) (layer F.SilkS)
