File: hardware/trs_pcb/trsmidi_input_8x.sch (KiCad schematic (older format))
At the start: 56 parts, among them J201 AudioJack3, J202 AudioJack3, J203 AudioJack3, J204 AudioJack3, J205 AudioJack3, J206 AudioJack3, J207 AudioJack3, J208 AudioJack3, U201 HCPL-2630, U202 HCPL-2630, U203 HCPL-2630, U204 HCPL-2630, U205 HCPL-2630, U206 HCPL-2630, U207 HCPL-2630, U208 HCPL-2630

Commit message: Add license hints to all hardware files
Other:
- note added: "Copyright (c) 2021 Florian Jung.\n\nThis source describes Open Hardware and is licensed under the CERN-OHL-S v2.\n\nYou may redistribute and modify this source and make products using it under\nthe terms of the CERN-OHL-S v2 (https://ohwr.org/cern_ohl_s_v2.txt).\n\nThis source is distributed WITHOUT ANY EXPRESS OR IMPLIED WARRANTY,\nINCLUDING OF MERCHANTABILITY, SATISFACTORY QUALITY AND FITNESS F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"
Changed lines of the file:
@@
 encoding utf-8
 Sheet 2 3
-Title ""
+Title "Midikraken TRS"
 Date ""
-Rev ""
-Comp ""
+Rev "01"
+Comp "Windfisch"
 Comment1 ""
 Comment2 ""
@@
 Wire Wire Line
 	5150 5550 4775 5550
+Text Notes 7950 6450 0    50   ~ 0
+Copyright (c) 2021 Florian Jung.\n\nThis source describes Open Hardware and is licensed under the CERN-OHL-S v2.\n\nYou may redistribute and modify this source and make products using it under\nthe terms of the CERN-OHL-S v2 (https://ohwr.org/cern_ohl_s_v2.txt).\n\nThis source is distributed WITHOUT ANY EXPRESS OR IMPLIED WARRANTY,\nINCLUDING OF MERCHANTABILITY, SATISFACTORY QUALITY AND FITNESS FOR A\nPARTICULAR PURPOSE. Please see the CERN-OHL-S v2 for applicable conditions.\n\nSource location: https://github.com/Windfisch/midikraken\n\nAs per CERN-OHL-S v2 section 4, should You produce hardware based on this\nsource, You must where practicable maintain the Source Location visible\non the external case of the Gizmo or other products you make using this\nsource.\n
 $EndSCHEMATC

Commit message: Bill of material
Parts:
- D201, D202, D203, D204, D205, D206, D207, D208: value LED -> red
- J201, J202, J203, J204, J205, J206, J207, J208: value AudioJack3 -> PJ324
Changed lines of the file:
@@
 AR Path="/60B37C5E/60B467EC" Ref="J201"  Part="1"
 F 0 "J201" H 982 1725 50  0000 C CNN
-F 1 "AudioJack3" H 982 1634 50  0000 C CNN
+F 1 "PJ324" H 982 1634 50  0000 C CNN
 F 2 "footprints:Jack_3.5mm_combo_ledino_upright" H 1000 1400 50  0001 C CNN
 F 3 "~" H 1000 1400 50  0001 C CNN
@@
 AR Path="/60B37C5E/60B4682F" Ref="D201"  Part="1"
 F 0 "D201" V 2639 857 50  0000 R CNN
-F 1 "LED" V 2548 857 50  0000 R CNN
+F 1 "red" V 2548 857 50  0000 R CNN
 F 2 "LED_THT:LED_D3.0mm_Horizontal_O6.35mm_Z2.0mm" H 2600 975 50  0001 C CNN
 F 3 "~" H 2600 975 50  0001 C CNN
@@
 AR Path="/60B37C5E/60B61B54" Ref="J202"  Part="1"
 F 0 "J202" H 982 3300 50  0000 C CNN
-F 1 "AudioJack3" H 982 3209 50  0000 C CNN
+F 1 "PJ324" H 982 3209 50  0000 C CNN
 F 2 "footprints:Jack_3.5mm_combo_ledino_upright" H 1000 2975 50  0001 C CNN
 F 3 "~" H 1000 2975 50  0001 C CNN
@@
 AR Path="/60B37C5E/60B61CCF" Ref="D202"  Part="1"
 F 0 "D202" V 2639 2432 50  0000 R CNN
-F 1 "LED" V 2548 2432 50  0000 R CNN
+F 1 "red" V 2548 2432 50  0000 R CNN
 F 2 "LED_THT:LED_D3.0mm_Horizontal_O6.35mm_Z2.0mm" H 2600 2550 50  0001 C CNN
 F 3 "~" H 2600 2550 50  0001 C CNN
@@
 AR Path="/60B37C5E/60B6B56B" Ref="J203"  Part="1"
 F 0 "J203" H 982 4875 50  0000 C CNN
-F 1 "AudioJack3" H 982 4784 50  0000 C CNN
+F 1 "PJ324" H 982 4784 50  0000 C CNN
 F 2 "footprints:Jack_3.5mm_combo_ledino_upright" H 1000 4550 50  0001 C CNN
 F 3 "~" H 1000 4550 50  0001 C CNN
@@
 	2400 4275 2400 4350
 Connection ~ 2400 4350
-$Comp
-L Device:LED D?
-U 1 1 60B6B7F2
-P 2600 4125
-AR Path="/60B6B7F2" Ref="D?"  Part="1"
-AR Path="/60B37C5E/60B6B7F2" Ref="D203"  Part="1"
-F 0 "D203" V 2639 4007 50  0000 R CNN
-F 1 "LED" V 2548 4007 50  0000 R CNN
-F 2 "LED_THT:LED_D3.0mm_Horizontal_O6.35mm_Z2.0mm" H 2600 4125 50  0001 C CNN
-F 3 "~" H 2600 4125 50  0001 C CNN
-	1    2600 4125
-	0    -1   -1   0
-$EndComp
 Wire Wire Line
 	2600 4575 2600 4750
@@
 AR Path="/60B37C5E/60B6B825" Ref="J204"  Part="1"
 F 0 "J204" H 982 6450 50  0000 C CNN
-F 1 "AudioJack3" H 982 6359 50  0000 C CNN
+F 1 "PJ324" H 982 6359 50  0000 C CNN
 F 2 "footprints:Jack_3.5mm_combo_ledino_upright" H 1000 6125 50  0001 C CNN
 F 3 "~" H 1000 6125 50  0001 C CNN
@@
 AR Path="/60B37C5E/60B6B87E" Ref="D204"  Part="1"
 F 0 "D204" V 2639 5582 50  0000 R CNN
-F 1 "LED" V 2548 5582 50  0000 R CNN
+F 1 "red" V 2548 5582 50  0000 R CNN
 F 2 "LED_THT:LED_D3.0mm_Horizontal_O6.35mm_Z2.0mm" H 2600 5700 50  0001 C CNN
 F 3 "~" H 2600 5700 50  0001 C CNN
@@
 AR Path="/60B37C5E/60B935FD" Ref="J205"  Part="1"
 F 0 "J205" H 3732 1725 50  0000 C CNN
-F 1 "AudioJack3" H 3732 1634 50  0000 C CNN
+F 1 "PJ324" H 3732 1634 50  0000 C CNN
 F 2 "footprints:Jack_3.5mm_combo_ledino_upright" H 3750 1400 50  0001 C CNN
 F 3 "~" H 3750 1400 50  0001 C CNN
@@
 AR Path="/60B37C5E/60B93A9C" Ref="D205"  Part="1"
 F 0 "D205" V 5389 857 50  0000 R CNN
-F 1 "LED" V 5298 857 50  0000 R CNN
+F 1 "red" V 5298 857 50  0000 R CNN
 F 2 "LED_THT:LED_D3.0mm_Horizontal_O6.35mm_Z2.0mm" H 5350 975 50  0001 C CNN
 F 3 "~" H 5350 975 50  0001 C CNN
@@
 AR Path="/60B37C5E/60B93ACE" Ref="J206"  Part="1"
 F 0 "J206" H 3732 3300 50  0000 C CNN
-F 1 "AudioJack3" H 3732 3209 50  0000 C CNN
+F 1 "PJ324" H 3732 3209 50  0000 C CNN
 F 2 "footprints:Jack_3.5mm_combo_ledino_upright" H 3750 2975 50  0001 C CNN
 F 3 "~" H 3750 2975 50  0001 C CNN
@@
 AR Path="/60B37C5E/60B93B27" Ref="D206"  Part="1"
 F 0 "D206" V 5389 2432 50  0000 R CNN
-F 1 "LED" V 5298 2432 50  0000 R CNN
+F 1 "red" V 5298 2432 50  0000 R CNN
 F 2 "LED_THT:LED_D3.0mm_Horizontal_O6.35mm_Z2.0mm" H 5350 2550 50  0001 C CNN
 F 3 "~" H 5350 2550 50  0001 C CNN
@@
 AR Path="/60B37C5E/60B93B59" Ref="J207"  Part="1"
 F 0 "J207" H 3732 4875 50  0000 C CNN
-F 1 "AudioJack3" H 3732 4784 50  0000 C CNN
+F 1 "PJ324" H 3732 4784 50  0000 C CNN
 F 2 "footprints:Jack_3.5mm_combo_ledino_upright" H 3750 4550 50  0001 C CNN
 F 3 "~" H 3750 4550 50  0001 C CNN
@@
 AR Path="/60B37C5E/60B93BB2" Ref="D207"  Part="1"
 F 0 "D207" V 5389 4007 50  0000 R CNN
-F 1 "LED" V 5298 4007 50  0000 R CNN
+F 1 "red" V 5298 4007 50  0000 R CNN
 F 2 "LED_THT:LED_D3.0mm_Horizontal_O6.35mm_Z2.0mm" H 5350 4125 50  0001 C CNN
 F 3 "~" H 5350 4125 50  0001 C CNN
@@
 AR Path="/60B37C5E/60B93BE4" Ref="J208"  Part="1"
 F 0 "J208" H 3732 6450 50  0000 C CNN
-F 1 "AudioJack3" H 3732 6359 50  0000 C CNN
+F 1 "PJ324" H 3732 6359 50  0000 C CNN
 F 2 "footprints:Jack_3.5mm_combo_ledino_upright" H 3750 6125 50  0001 C CNN
 F 3 "~" H 3750 6125 50  0001 C CNN
@@
 AR Path="/60B37C5E/60B93C3D" Ref="D208"  Part="1"
 F 0 "D208" V 5389 5582 50  0000 R CNN
-F 1 "LED" V 5298 5582 50  0000 R CNN
+F 1 "red" V 5298 5582 50  0000 R CNN
 F 2 "LED_THT:LED_D3.0mm_Horizontal_O6.35mm_Z2.0mm" H 5350 5700 50  0001 C CNN
 F 3 "~" H 5350 5700 50  0001 C CNN
@@
 Text Notes 7950 6450 0    50   ~ 0
 Copyright (c) 2021 Florian Jung.\n\nThis source describes Open Hardware and is licensed under the CERN-OHL-S v2.\n\nYou may redistribute and modify this source and make products using it under\nthe terms of the CERN-OHL-S v2 (https://ohwr.org/cern_ohl_s_v2.txt).\n\nThis source is distributed WITHOUT ANY EXPRESS OR IMPLIED WARRANTY,\nINCLUDING OF MERCHANTABILITY, SATISFACTORY QUALITY AND FITNESS FOR A\nPARTICULAR PURPOSE. Please see the CERN-OHL-S v2 for applicable conditions.\n\nSource location: https://github.com/Windfisch/midikraken\n\nAs per CERN-OHL-S v2 section 4, should You produce hardware based on this\nsource, You must where practicable maintain the Source Location visible\non the external case of the Gizmo or other products you make using this\nsource.\n
+$Comp
+L Device:LED D?
+U 1 1 60B6B7F2
+P 2600 4125
+AR Path="/60B6B7F2" Ref="D?"  Part="1"
+AR Path="/60B37C5E/60B6B7F2" Ref="D203"  Part="1"
+F 0 "D203" V 2639 4007 50  0000 R CNN
+F 1 "red" V 2548 4007 50  0000 R CNN
+F 2 "LED_THT:LED_D3.0mm_Horizontal_O6.35mm_Z2.0mm" H 2600 4125 50  0001 C CNN
+F 3 "~" H 2600 4125 50  0001 C CNN
+	1    2600 4125
+	0    -1   -1   0
+$EndComp
 $EndSCHEMATC
