File: hardware/trs_pcb/trs_midi_output_8x.sch (KiCad schematic (older format))
At the start: 56 parts, among them J301 AudioJack3, J302 AudioJack3, J303 AudioJack3, J304 AudioJack3, J305 AudioJack3, J306 AudioJack3, J307 AudioJack3, J308 AudioJack3

Commit message: Add license hints to all hardware files
Other:
- note added: "Copyright (c) 2021 Florian Jung.\n\nThis source describes Open Hardware and is licensed under the CERN-OHL-S v2.\n\nYou may redistribute and modify this source and make products using it under\nthe terms of the CERN-OHL-S v2 (https://ohwr.org/cern_ohl_s_v2.txt).\n\nThis source is distributed WITHOUT ANY EXPRESS OR IMPLIED WARRANTY,\nINCLUDING OF MERCHANTABILITY, SATISFACTORY QUALITY AND FITNESS F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"
Changed lines of the file:
@@
 encoding utf-8
 Sheet 3 3
-Title ""
+Title "Midikraken TRS"
 Date ""
-Rev ""
-Comp ""
+Rev "01"
+Comp "Windfisch"
 Comment1 ""
 Comment2 ""
@@
 Wire Wire Line
 	4125 5275 4225 5275
+Text Notes 725  7500 0    50   ~ 0
+Copyright (c) 2021 Florian Jung.\n\nThis source describes Open Hardware and is licensed under the CERN-OHL-S v2.\n\nYou may redistribute and modify this source and make products using it under\nthe terms of the CERN-OHL-S v2 (https://ohwr.org/cern_ohl_s_v2.txt).\n\nThis source is distributed WITHOUT ANY EXPRESS OR IMPLIED WARRANTY,\nINCLUDING OF MERCHANTABILITY, SATISFACTORY QUALITY AND FITNESS FOR A\nPARTICULAR PURPOSE. Please see the CERN-OHL-S v2 for applicable conditions.\n\nSource location: https://github.com/Windfisch/midikraken\n\nAs per CERN-OHL-S v2 section 4, should You produce hardware based on this\nsource, You must where practicable maintain the Source Location visible\non the external case of the Gizmo or other products you make using this\nsource.\n
 $EndSCHEMATC

Commit message: Bill of material
Parts:
- J301, J302, J303, J304, J305, J306, J307, J308: value AudioJack3 -> PJ324
Changed lines of the file:
@@
 P 2050 1625
 F 0 "J301" H 1800 1650 50  0000 R CNN
-F 1 "AudioJack3" H 2175 1350 50  0000 R CNN
+F 1 "PJ324" H 2175 1350 50  0000 R CNN
 F 2 "footprints:Jack_3.5mm_combo_ledino_upright" H 2050 1625 50  0001 C CNN
 F 3 "~" H 2050 1625 50  0001 C CNN
@@
 P 2050 2875
 F 0 "J302" H 1800 2900 50  0000 R CNN
-F 1 "AudioJack3" H 2175 2600 50  0000 R CNN
+F 1 "PJ324" H 2175 2600 50  0000 R CNN
 F 2 "footprints:Jack_3.5mm_combo_ledino_upright" H 2050 2875 50  0001 C CNN
 F 3 "~" H 2050 2875 50  0001 C CNN
@@
 P 2050 4125
 F 0 "J303" H 1800 4150 50  0000 R CNN
-F 1 "AudioJack3" H 2175 3850 50  0000 R CNN
+F 1 "PJ324" H 2175 3850 50  0000 R CNN
 F 2 "footprints:Jack_3.5mm_combo_ledino_upright" H 2050 4125 50  0001 C CNN
 F 3 "~" H 2050 4125 50  0001 C CNN
@@
 P 2050 5375
 F 0 "J304" H 1800 5400 50  0000 R CNN
-F 1 "AudioJack3" H 2175 5100 50  0000 R CNN
+F 1 "PJ324" H 2175 5100 50  0000 R CNN
 F 2 "footprints:Jack_3.5mm_combo_ledino_upright" H 2050 5375 50  0001 C CNN
 F 3 "~" H 2050 5375 50  0001 C CNN
@@
 P 4425 1625
 F 0 "J305" H 4175 1650 50  0000 R CNN
-F 1 "AudioJack3" H 4550 1350 50  0000 R CNN
+F 1 "PJ324" H 4550 1350 50  0000 R CNN
 F 2 "footprints:Jack_3.5mm_combo_ledino_upright" H 4425 1625 50  0001 C CNN
 F 3 "~" H 4425 1625 50  0001 C CNN
@@
 P 4425 2875
 F 0 "J306" H 4175 2900 50  0000 R CNN
-F 1 "AudioJack3" H 4550 2600 50  0000 R CNN
+F 1 "PJ324" H 4550 2600 50  0000 R CNN
 F 2 "footprints:Jack_3.5mm_combo_ledino_upright" H 4425 2875 50  0001 C CNN
 F 3 "~" H 4425 2875 50  0001 C CNN
@@
 P 4425 4125
 F 0 "J307" H 4175 4150 50  0000 R CNN
-F 1 "AudioJack3" H 4550 3850 50  0000 R CNN
+F 1 "PJ324" H 4550 3850 50  0000 R CNN
 F 2 "footprints:Jack_3.5mm_combo_ledino_upright" H 4425 4125 50  0001 C CNN
 F 3 "~" H 4425 4125 50  0001 C CNN
@@
 P 4425 5375
 F 0 "J308" H 4175 5400 50  0000 R CNN
-F 1 "AudioJack3" H 4550 5100 50  0000 R CNN
+F 1 "PJ324" H 4550 5100 50  0000 R CNN
 F 2 "footprints:Jack_3.5mm_combo_ledino_upright" H 4425 5375 50  0001 C CNN
 F 3 "~" H 4425 5375 50  0001 C CNN

Commit message: Change LED resistors from 1k to 220 Ohm.
Closes #61.
Parts:
- R301, R302, R303, R304, R305, R306, R307, R308, R317, R318, R319, R320, R321, R322, R323, R324: value 1k -> 220
Changed lines of the file:
@@
 P 1150 1050
 F 0 "R301" H 950 1100 50  0000 L CNN
-F 1 "1k" V 1150 1000 50  0000 L CNN
+F 1 "220" V 1150 1000 50  0000 L CNN
 F 2 "Resistor_SMD:R_0805_2012Metric" V 1080 1050 50  0001 C CNN
 F 3 "~" H 1150 1050 50  0001 C CNN
@@
 P 1350 1050
 F 0 "R305" H 1420 1096 50  0000 L CNN
-F 1 "1k" V 1350 1000 50  0000 L CNN
+F 1 "220" V 1350 1000 50  0000 L CNN
 F 2 "Resistor_SMD:R_0805_2012Metric" V 1280 1050 50  0001 C CNN
 F 3 "~" H 1350 1050 50  0001 C CNN
@@
 P 1150 2300
 F 0 "R302" H 950 2350 50  0000 L CNN
-F 1 "1k" V 1150 2250 50  0000 L CNN
+F 1 "220" V 1150 2250 50  0000 L CNN
 F 2 "Resistor_SMD:R_0805_2012Metric" V 1080 2300 50  0001 C CNN
 F 3 "~" H 1150 2300 50  0001 C CNN
@@
 P 1350 2300
 F 0 "R306" H 1420 2346 50  0000 L CNN
-F 1 "1k" V 1350 2250 50  0000 L CNN
+F 1 "220" V 1350 2250 50  0000 L CNN
 F 2 "Resistor_SMD:R_0805_2012Metric" V 1280 2300 50  0001 C CNN
 F 3 "~" H 1350 2300 50  0001 C CNN
@@
 P 1150 3550
 F 0 "R303" H 950 3600 50  0000 L CNN
-F 1 "1k" V 1150 3500 50  0000 L CNN
+F 1 "220" V 1150 3500 50  0000 L CNN
 F 2 "Resistor_SMD:R_0805_2012Metric" V 1080 3550 50  0001 C CNN
 F 3 "~" H 1150 3550 50  0001 C CNN
@@
 P 1350 3550
 F 0 "R307" H 1420 3596 50  0000 L CNN
-F 1 "1k" V 1350 3500 50  0000 L CNN
+F 1 "220" V 1350 3500 50  0000 L CNN
 F 2 "Resistor_SMD:R_0805_2012Metric" V 1280 3550 50  0001 C CNN
 F 3 "~" H 1350 3550 50  0001 C CNN
@@
 P 1150 4800
 F 0 "R304" H 950 4850 50  0000 L CNN
-F 1 "1k" V 1150 4750 50  0000 L CNN
+F 1 "220" V 1150 4750 50  0000 L CNN
 F 2 "Resistor_SMD:R_0805_2012Metric" V 1080 4800 50  0001 C CNN
 F 3 "~" H 1150 4800 50  0001 C CNN
@@
 P 1350 4800
 F 0 "R308" H 1420 4846 50  0000 L CNN
-F 1 "1k" V 1350 4750 50  0000 L CNN
+F 1 "220" V 1350 4750 50  0000 L CNN
 F 2 "Resistor_SMD:R_0805_2012Metric" V 1280 4800 50  0001 C CNN
 F 3 "~" H 1350 4800 50  0001 C CNN
@@
 P 3525 1050
 F 0 "R317" H 3325 1100 50  0000 L CNN
-F 1 "1k" V 3525 1000 50  0000 L CNN
+F 1 "220" V 3525 1000 50  0000 L CNN
 F 2 "Resistor_SMD:R_0805_2012Metric" V 3455 1050 50  0001 C CNN
 F 3 "~" H 3525 1050 50  0001 C CNN
@@
 P 3725 1050
 F 0 "R321" H 3795 1096 50  0000 L CNN
-F 1 "1k" V 3725 1000 50  0000 L CNN
+F 1 "220" V 3725 1000 50  0000 L CNN
 F 2 "Resistor_SMD:R_0805_2012Metric" V 3655 1050 50  0001 C CNN
 F 3 "~" H 3725 1050 50  0001 C CNN
@@
 P 3525 2300
 F 0 "R318" H 3325 2350 50  0000 L CNN
-F 1 "1k" V 3525 2250 50  0000 L CNN
+F 1 "220" V 3525 2250 50  0000 L CNN
 F 2 "Resistor_SMD:R_0805_2012Metric" V 3455 2300 50  0001 C CNN
 F 3 "~" H 3525 2300 50  0001 C CNN
@@
 P 3725 2300
 F 0 "R322" H 3795 2346 50  0000 L CNN
-F 1 "1k" V 3725 2250 50  0000 L CNN
+F 1 "220" V 3725 2250 50  0000 L CNN
 F 2 "Resistor_SMD:R_0805_2012Metric" V 3655 2300 50  0001 C CNN
 F 3 "~" H 3725 2300 50  0001 C CNN
@@
 P 3525 3550
 F 0 "R319" H 3325 3600 50  0000 L CNN
-F 1 "1k" V 3525 3500 50  0000 L CNN
+F 1 "220" V 3525 3500 50  0000 L CNN
 F 2 "Resistor_SMD:R_0805_2012Metric" V 3455 3550 50  0001 C CNN
 F 3 "~" H 3525 3550 50  0001 C CNN
@@
 P 3725 3550
 F 0 "R323" H 3795 3596 50  0000 L CNN
-F 1 "1k" V 3725 3500 50  0000 L CNN
+F 1 "220" V 3725 3500 50  0000 L CNN
 F 2 "Resistor_SMD:R_0805_2012Metric" V 3655 3550 50  0001 C CNN
 F 3 "~" H 3725 3550 50  0001 C CNN
@@
 P 3525 4800
 F 0 "R320" H 3325 4850 50  0000 L CNN
-F 1 "1k" V 3525 4750 50  0000 L CNN
+F 1 "220" V 3525 4750 50  0000 L CNN
 F 2 "Resistor_SMD:R_0805_2012Metric" V 3455 4800 50  0001 C CNN
 F 3 "~" H 3525 4800 50  0001 C CNN
@@
 P 3725 4800
 F 0 "R324" H 3795 4846 50  0000 L CNN
-F 1 "1k" V 3725 4750 50  0000 L CNN
+F 1 "220" V 3725 4750 50  0000 L CNN
 F 2 "Resistor_SMD:R_0805_2012Metric" V 3655 4800 50  0001 C CNN
 F 3 "~" H 3725 4800 50  0001 C CNN
